File: Control_PCB/mcu.kicad_sch (KiCad schematic)
At the start: 8 parts, among them U1 STM32G473VET3

Commit message: 02-10-2026
Connections:
- net CAN_STB: now reaches U1.61 (PD14)
- net CAN_FAULT: now reaches U1.9 (PC15-OSC32_OUT)
- net CAN_ENA: now reaches U1.96 (PB9)
Changed lines of the file:
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@@
+	(wire
+		(pts
+			(xy 124.46 68.58) (xy 137.16 68.58)
+		)
+		(stroke
+			(width 0)
+			(type default)
+		)
+	)
 	(wire
 		(pts
@@
 	(wire
 		(pts
-			(xy 43.18 60.96) (xy 53.34 60.96)
+			(xy 40.64 60.96) (xy 53.34 60.96)
 		)
 		(stroke
@@
 	(wire
 		(pts
+			(xy 40.64 96.52) (xy 53.34 96.52)
+		)
+		(stroke
+			(width 0)
+			(type default)
+		)
+	)
+	(wire
+		(pts
 			(xy 85.09 181.61) (xy 88.9 181.61)
 		)
@@
 	(wire
 		(pts
-			(xy 43.18 58.42) (xy 53.34 58.42)
+			(xy 40.64 58.42) (xy 53.34 58.42)
 		)
 		(stroke
@@
 		(pts
 			(xy 121.92 158.75) (xy 115.57 158.75)
+		)
+		(stroke
+			(width 0)
+			(type default)
+		)
+	)
+	(wire
+		(pts
+			(xy 124.46 109.22) (xy 137.16 109.22)
 		)
 		(stroke
@@
 		)
 	)
-	(label "ENA_INRUSH"
-		(at 137.16 91.44 180)
-		(effects
-			(font
-				(size 1.27 1.27)
-			)
-			(justify right bottom)
-		)
-	)
 	(label "AD_5V"
 		(at 40.64 76.2 0)
@@
 	(hierarchical_label "CAN_TX"
 		(shape output)
-		(at 43.18 60.96 180)
-		(effects
-			(font
-				(size 1.27 1.27)
+		(at 40.64 60.96 180)
+		(effects
+			(font
+				(size 1.27 1.27)
+			)
+			(justify right)
+		)
+	)
+	(hierarchical_label "ENA_INRUSH"
+		(shape output)
+		(at 137.16 91.44 0)
+		(effects
+			(font
+				(size 1.27 1.27)
+			)
+			(justify left)
+		)
+	)
+	(hierarchical_label "CAN_STB"
+		(shape output)
+		(at 137.16 109.22 0)
+		(effects
+			(font
+				(size 1.27 1.27)
+				(thickness 0.1588)
+			)
+			(justify left)
+		)
+	)
+	(hierarchical_label "CAN_FAULT"
+		(shape input)
+		(at 137.16 68.58 0)
+		(effects
+			(font
+				(size 1.27 1.27)
+				(thickness 0.1588)
+			)
+			(justify left)
+		)
+	)
+	(hierarchical_label "CAN_ENA"
+		(shape output)
+		(at 40.64 96.52 180)
+		(effects
+			(font
+				(size 1.27 1.27)
+				(thickness 0.1588)
 			)
 			(justify right)
@@
 	(hierarchical_label "CAN_RX"
 		(shape input)
-		(at 43.18 58.42 180)
-		(effects
-			(font
+		(at 40.64 58.42 180)
+		(effects
+			(font

Commit message: 07-20-2026
Parts:
- added C49, C50: 24p, Capacitor_SMD:C_0603_1608Metric, symbol Device:C_Small
- added C51: 1u, Capacitor_SMD:C_0603_1608Metric, symbol Device:C_Small
- added C52: 10n, Capacitor_SMD:C_0603_1608Metric, symbol Device:C_Small
- added D21: PESD5V2S2UT, Package_TO_SOT_SMD:SOT-23, symbol Device:D_Zener_Dual_CommonAnode_KKA
- added J4: Micro Match, Connector_Molex:Molex_Mini-Fit_Jr_5569-06A2_2x03_P4.20mm_Horizontal, symbol Connector_Generic:Conn_02x03_Counter_Clockwise
- added R63, R64: 100, symbol Device:R_Small
- added R65: 470k, symbol Device:R_Small
- added R66: 15k, symbol Device:R_Small
- added R67: 100k, Resistor_SMD:R_0603_1608Metric, symbol Device:R_Small
- added R68: 10k, symbol Device:R_Small
- added TP19, TP20, TP21, TP22: TestPoint, TestPoint:TestPoint_Pad_D1.5mm, symbol Connector:TestPoint
- added Y1: ABM3BAIG, Crystal:Crystal_SMD_5032-4Pin_5.0x3.2mm, symbol Device:Crystal_GND24
Connections:
- net +3V3: now also J4.5 (Pin_5), R68.2
- net GND: now also C49.2, C50.2, C51.1, C52.1, D21.3 (A), J4.2 (Pin_2), R65.1, R67.1, Y1.2 (G), Y1.4 (G)
- net PROG_BOOT: now also C51.2, R66.2, R67.2
- net PROG_RX: now also D21.2 (K), R63.2, R66.1, TP21.1
- net PROG_TX: now also D21.1 (K), R64.2, R65.2, TP22.1
- net SWD_CLK: now also J4.3 (Pin_3)
- net SWD_IO: now also J4.1 (Pin_1)
- net AD_12V: now reaches U1.21 (PA1)
- net AD_GPIO1: now reaches U1.22 (PA2)
- net AD_GPIO2: now reaches U1.25 (PA3)
- net AD_GPIO3: now reaches U1.26 (PA4)
- net AD_TEMP_INRUSH: now reaches U1.27 (PA5)
- net AD_TEMP_AMB: now reaches U1.28 (PA6)
- net AD_VCC_CURRENT: now reaches U1.29 (PA7)
- net LIN_PULLDOWN: now reaches U1.34 (PB2)
- net LIN_TX: now reaches U1.55 (PD8)
- net LIN_RX: now reaches U1.56 (PD9)
- net ENA_LIN_MASTER: now reaches U1.62 (PD15)
- net LIN_SLEEP: now reaches U1.69 (PA8)
- net at U1.12 (PF0-OSC_IN): now also C49.1, Y1.1
- net at U1.13 (PF1-OSC_OUT): now also C50.1, Y1.3
- net ~{RST}: now reaches U1.14 (PG10-NRST)
- net ~{RST}: now also C52.2, J4.4 (Pin_4), R68.1
- net JTRST: no longer names the net of U1.91 (PB4)
- net SWO/JTDO renamed SWO
- net SWO: now also J4.6 (Pin_6)
- new net: R64.1, TP20.1
- new net: R63.1, TP19.1
Other:
- note added: "CON_PROG_RX"
- note added: "CON_PROG_TX"
- note added: "PROG 6-pin!!"
- note added: "UART"
- moved on the sheet: C1, C2, C3, C4, C5, C6, C7, U1A, U1B

Commit message: 10-10-2026
Connections:
- net HEART_BEAT renamed HEARTBEAT_mcu
Other:
- moved on the sheet: C49, C50, C51, D21, J4, R65, R66, R67, TP19, TP20, TP22, U1A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

Commit message: Before removing stuffs
Parts:
- J4: footprint Connector_Molex:Molex_Mini-Fit_Jr_5569-06A2_2x03_P4.20mm_Horizontal -> Control_PCB:CONN6_7-188275-6_TEC
- R63, R64, R65, R66, R68: footprint (none) -> Resistor_SMD:R_0603_1608Metric
Changed lines of the file:
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@@
 			)
 		)
-		(property "Footprint" "Connector_Molex:Molex_Mini-Fit_Jr_5569-06A2_2x03_P4.20mm_Horizontal"
+		(property "Footprint" "Control_PCB:CONN6_7-188275-6_TEC"
 			(at 232.41 105.41 0)
 			(hide yes)
@@
 			)
 		)
-		(property "Footprint" ""
+		(property "Footprint" "Resistor_SMD:R_0603_1608Metric"
 			(at 213.36 143.51 0)
 			(hide yes)
@@
 			)
 		)
-		(property "Footprint" ""
+		(property "Footprint" "Resistor_SMD:R_0603_1608Metric"
 			(at 251.46 130.81 0)
 			(hide yes)
@@
 			)
 		)
-		(property "Footprint" ""
+		(property "Footprint" "Resistor_SMD:R_0603_1608Metric"
 			(at 227.33 34.29 0)
 			(hide yes)
@@
 			)
 		)
-		(property "Footprint" ""
+		(property "Footprint" "Resistor_SMD:R_0603_1608Metric"
 			(at 241.3 147.32 0)
 			(hide yes)
@@
 			)
 		)
-		(property "Footprint" ""
+		(property "Footprint" "Resistor_SMD:R_0603_1608Metric"
 			(at 213.36 134.62 0)
 			(hide yes)

Commit message: 15-10-2026
Connections:
- net AD_GPIO4: now reaches U1.30 (PC4)
- net AD_VCC: now reaches U1.31 (PC5)
- net LED_BLUE: now reaches U1.58 (PD11)
- net LED_RED: now reaches U1.68 (PC9)
- net LED_GREEN: now reaches U1.46 (PE15)
- no-connect marks 0 -> 45

Commit message: Schematics mostly done
Parts:
- added C212, C214: 100n, Capacitor_SMD:C_0603_1608Metric, symbol Device:C_Small
- added C213, C215: 1u, Capacitor_SMD:C_0603_1608Metric, symbol Device:C_Small
- added FB201: FerriteBead_Small, Inductor_SMD:L_0603_1608Metric, symbol Device:FerriteBead_Small
- added R207: 47, Resistor_SMD:R_0603_1608Metric, symbol Device:R_Small
- C204: renamed from C1; value 10u -> 22u; footprint Capacitor_SMD:C_0603_1608Metric -> Capacitor_SMD:C_0805_2012Metric
- R203: renamed from R63; value 100 -> 120
- R205: renamed from R64; value 100 -> 120
- renumbered C49 to C201, C50 to C202, C52 to C203, C2 to C205, C3 to C206, C4 to C207, C5 to C208, C6 to C209, C7 to C210, C51 to C211, D21 to D201, J4 to J201, R68 to R201, R66 to R202, R67 to R204, R65 to R206, TP19 to TP201, TP21 to TP202, TP20 to TP203, TP22 to TP204, U1 to U201, Y1 to Y201
Connections:
- net +3V3: now also FB201.2
- net +3V3_VDDA: now also C212.1, C213.1, FB201.1, R207.1
- net GND: now also C212.2, C213.2, C214.2, C215.2
- net at U201.36 (VREF+): now also C214.1, C215.1, R207.2
Other:
- note added: "AN2586"
- note removed: "ADD VDDA Filter"
- moved on the sheet: C201, C202, C203, C204, C205, C206, C207, C208, C209, C210, R201, U201B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
