File: Control_PCB/IO_Interface.kicad_sch (KiCad schematic)
At the start: 9 parts, among them U6 TCAN1043xDxQ1

Commit message: 04-10-2026
Parts:
- added C40, C41, C42, C43: 1n, Capacitor_SMD:C_0603_1608Metric, symbol Device:C_Small
- added C44, C45, C46, C47: 100n, Package_SO:SOIC-16_3.9x9.9mm_P1.27mm, symbol Device:C_Small
- added D10, D8: BAV99, Package_TO_SOT_SMD:SOT-23, symbol Diode:BAV99
- added D11, D4, D6, D9: MM3Z62VB, Diode_SMD:D_SOD-323F, symbol Diode:MM3Zxx
- added E1, E2, E3, E4, E5, E6: SparkGap, LED_SMD:LED_Kingbright_APFA3010_3x1.5mm_Horizontal, symbol Device:SparkGap
- added L4, L5, L6, L7: L_Small, Package_DFN_QFN:UQFN-20-1EP_3x3mm_P0.4mm_EP1.7x1.7mm_ThermalVias, symbol Device:L_Small
- added Q10, Q11, Q4, Q7: BCX56, Package_TO_SOT_SMD:SOT-89-3, symbol Transistor_BJT:BCX56
- added Q12, Q13, Q6, Q8: BC846, Package_TO_SOT_SMD:SOT-23, symbol Transistor_BJT:BC846
- added Q9: PUMH11, Package_TO_SOT_SMD:SOT-363_SC-70-6, symbol Transistor_BJT:PUMX1
- added R20, R21, R26, R27, R30, R31, R40, R42: 18k, Resistor_SMD:R_0603_1608Metric, symbol Device:R_Small
- added R24, R28, R32, R44: 100k, Resistor_SMD:R_0603_1608Metric, symbol Device:R_Small
- added R25, R29, R33, R45: 4k7, Resistor_SMD:R_0603_1608Metric, symbol Device:R_Small
- added R34, R36, R38, R39: 47, Resistor_SMD:R_0603_1608Metric, symbol Device:R_Small
- added R35, R43: 10k, Resistor_SMD:R_0603_1608Metric, symbol Device:R_Small
- added R37, R41: 68k, Resistor_SMD:R_0603_1608Metric, symbol Device:R_Small
- added RV1, RV2, RV3, RV4: MAV0010DP, symbol Device:Varistor
- added TP10, TP11, TP12, TP13, TP6, TP7, TP8, TP9: TestPoint, TestPoint:TestPoint_Pad_D1.5mm, symbol Connector:TestPoint
Connections:
- net CANH: now also E6.2
- net CANL: now also E5.2
- net GND: now also C40.1, C41.1, C42.1, C43.1, C44.2, C45.2, C46.2, C47.2, D11.2 (A), D4.2 (A), D6.2 (A), D9.2 (A), E1.1, E2.1, E3.1, E4.1, Q13.2 (E), Q6.2 (E), Q9.1 (E1), Q9.4 (E2), R25.1, R29.1, R33.1, R34.1, R39.1, R45.1, RV1.2, RV2.2, RV3.2, RV4.2
- new net: R30.2, R31.1
- new net: C42.2, D9.1 (K), R31.2, R32.1
- new net: Q4.1 (B), Q6.3 (C), R35.1
- new net: D8.2 (A), Q4.2 (C)
- new net: Q4.3 (E), Q6.1 (B), R34.2
- new net: Q7.1 (B), Q8.2 (E), R37.1
- new net: Q7.2 (C), Q8.1 (B), R36.1
- new net: D8.1 (K), Q7.3 (E)
- new net: C43.2, D11.1 (K), R42.2, R44.1
- new net: Q8.3 (C), R36.2
- new net: R20.2, R21.1
- new net: R40.2, R42.1
- new net: Q11.1 (B), Q13.3 (C), R43.1
- new net: D10.2 (A), Q11.2 (C)
- new net: Q11.3 (E), Q13.1 (B), R39.2
- new net: D10.1 (K), Q10.3 (E)
- new net: Q10.2 (C), Q12.1 (B), R38.1
- new net: Q10.1 (B), Q12.2 (E), R41.1
- new net: Q12.3 (C), R38.2
- new net: C40.2, D4.1 (K), R21.2, R24.1
- new net: Q9.6 (C1), R37.2
- new net: C41.2, D6.1 (K), R27.2, R28.1
- new net: R26.2, R27.1
- new net: Q9.3 (C2), R41.2
- new net AD_GPIO1: R24.2, R25.2, TP7.1
- new net AD_GPIO2: R28.2, R29.2, TP9.1
- new net AD_GPIO3: R32.2, R33.2, TP11.1
- new net AD_GPIO4: R44.2, R45.2, TP13.1
- new net GPIO1: E1.2, L4.1
- new net GPIO2: E2.2, L5.1
- new net GPIO3: E4.2, L6.1
- new net GPIO3_HI: Q9.2 (B1)
- new net GPIO3_LO: R35.2
- new net GPIO4: E3.2, L7.1
- new net GPIO4_HI: Q9.5 (B2)
- new net GPIO4_LO: R43.2
- new net GPIO_1: C44.1, L4.2, R20.1, RV1.1, TP6.1
- new net GPIO_2: C45.1, L5.2, R26.1, RV2.1, TP8.1
- new net GPIO_3: C46.1, D8.3 (K), L6.2, R30.1, RV3.1, TP10.1
- new net GPIO_4: C47.1, D10.3 (K), L7.2, R40.1, RV4.1, TP12.1
Other:
- note added: "GPIO - Input Filtering"
- note added: "GPIO 3"
- note added: "INPUT 1"
- moved on the sheet: C36, C37, C38, C39, R18, R19, TP4, TP5, U6

Commit message: 07-20-2026
Parts:
- removed L4, L5, L6, L7: L_Small, Package_DFN_QFN:UQFN-20-1EP_3x3mm_P0.4mm_EP1.7x1.7mm_ThermalVias, symbol Device:L_Small
- removed RV1, RV2, RV3, RV4: MAV0010DP, symbol Device:Varistor
- added C48: 100n, Capacitor_SMD:C_0603_1608Metric, symbol Device:C_Small
- added D12, D13, D14, D15: SMAJ58A, Diode_SMD:D_SMA, symbol Diode:SMAJ58A
- added D16: ESD2CANFD60-Q1, Package_TO_SOT_SMD:SOT-23-3, symbol Device:D_TVS_Dual_AAC
- added D19: BAS516, Diode_SMD:D_SOD-523, symbol Diode:BAS516
- added L4: DR331-513AE, Inductor_SMD:L_CommonMode_Bourns_DR331, symbol Device:L_Coupled_1423
- added R46, R47, R48, R49: 100, Resistor_SMD:R_1206_3216Metric, symbol Device:R_Small
- added R56: 47k, symbol Device:R_Small
- added R61: 100k, symbol Device:R_Small
- added R62: 10k, symbol Device:R_Small
- added TP18, TP23: TestPoint, TestPoint:TestPoint_Pad_D1.5mm, symbol Connector:TestPoint
- added U7: (no value), symbol Control_PCB:TLIN2021
- C44, C45, C46, C47: footprint Package_SO:SOIC-16_3.9x9.9mm_P1.27mm -> (none)
- E1, E2, E3, E4, E5, E6: footprint LED_SMD:LED_Kingbright_APFA3010_3x1.5mm_Horizontal -> Control_PCB:Sparkgap_2021-09-02
Connections:
- net +3V3: now also R61.1, R62.2
- net CANH: now also D16.1 (A1), L4.1; no longer R18.1, TP4.1, U6.13 (CANH)
- net CANL: now also D16.2 (A2), L4.2; no longer R19.2, TP5.1, U6.12 (CANL)
- net GND: now also E5.1, E6.1, C48.2, D12.2 (A2), D13.2 (A2), D14.2 (A2), D15.2 (A2), D16.3 (common), U7.5 (GND), U7.9 (PAD)
- net GPIO1: now also D12.1 (A1), R46.2
- net GPIO2: now also D13.1 (A1), R47.2
- net GPIO3: now also D14.1 (A1), R48.2
- net GPIO4: now also D15.1 (A1), R49.2
- net GPIO_1: now also R46.1
- net GPIO_2: now also R47.1
- net GPIO_3: now also R48.1
- net GPIO_4: now also R49.1
- new net: L4.3, R19.2, TP5.1, U6.12 (CANL)
- new net: L4.4, R18.1, TP4.1, U6.13 (CANH)
- new net: C48.1, D19.1 (K), R56.1, U7.7 (V_Sup)
- new net: R56.2, U7.3 (WAKE)
- new net +12V: D19.2 (A)
- new net LIN: TP23.1, U7.6 (LIN)
- new net LIN_RX: R62.1, U7.1 (RxD)
- new net LIN_SLEEP: TP18.1, U7.2 (EN)
- new net LIN_TX: R61.2, U7.4 (TxD)
- no-connect marks 1 -> 2
Other:
- note added: "Add Pull Down AND LIN Master Circuits!"
- note added: "GPIO - Input Protection"
- note added: "LIN"
- note removed: "GPIO - Input Filtering"
- moved on the sheet: C36, C37, C38, C39, C44, C45, C46, C47, E5, E6, R18, R19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

Commit message: 10-10-2026
Parts:
- added C53: C_Small, Package_LCC:PLCC-44_16.6x16.6mm_P1.27mm, symbol Device:C_Small
- added D20: SMAJ16A, Diode_SMD:D_SMA, symbol Diode:SMAJ58A
- added Q14: BCX56, Package_TO_SOT_SMD:SOT-89-3, symbol Transistor_BJT:BCX56
- added R69: 1k, Resistor_SMD:R_0603_1608Metric, symbol Device:R_Small
- added R70, R71, R72: 100k, Resistor_SMD:R_0603_1608Metric, symbol Device:R_Small
Connections:
- net +12V: now also R71.2
- net GND: now also C53.2, D20.2 (A2), Q14.3 (E), R70.1
- new net: Q14.1 (B), R69.1, R70.2
- new net: Q14.2 (C), R71.1, R72.1
- new net HEARTBEAT: C53.1, D20.1 (A1), R72.2
- new net HEARTBEAT_mcu: R69.2

Commit message: Before removing stuffs
Parts:
- C44, C45, C46, C47: footprint (none) -> Capacitor_SMD:C_0603_1608Metric
- C53: value C_Small -> 100n; footprint Package_LCC:PLCC-44_16.6x16.6mm_P1.27mm -> Capacitor_SMD:C_0603_1608Metric
- R56, R61, R62: footprint (none) -> Resistor_SMD:R_0603_1608Metric
- U7: value (none) -> TLIN2021; footprint (none) -> Package_SO:SOIC-8_5.3x5.3mm_P1.27mm
Connections:
- net CANH: now also L4.2; no longer L4.1
- net CANL: now also L4.1; no longer L4.2
- net at R19.2, TP5.1, U6.12 (CANL): now also L4.4; no longer L4.3
- net at R18.1, TP4.1, U6.13 (CANH): now also L4.3; no longer L4.4
Other:
- note added: "INPUT 2"
Changed lines of the file:
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@@
 		)
 	)
-	(text "INPUT 1"
+	(text "INPUT 2"
 		(exclude_from_sim no)
 		(at 25.146 109.982 0)
@@
 		(lib_id "Device:L_Coupled_1423")
 		(at 54.61 170.815 0)
+		(mirror x)
 		(unit 1)
 		(body_style 1)
@@
 		(in_pos_files yes)
 		(dnp no)
-		(fields_autoplaced yes)
 		(property "Reference" "L4"
-			(at 54.229 163.195 0)
+			(at 54.229 178.435 0)
 			(show_name no)
 			(do_not_autoplace no)
@@
 		)
 		(property "Value" "DR331-513AE"
-			(at 54.229 165.735 0)
+			(at 54.229 175.895 0)
 			(show_name no)
 			(do_not_autoplace no)
@@
 			)
 		)
-		(property "Footprint" ""
+		(property "Footprint" "Resistor_SMD:R_0603_1608Metric"
 			(at 255.27 46.99 0)
 			(hide yes)
@@
 			)
 		)
-		(property "Footprint" ""
+		(property "Footprint" "Capacitor_SMD:C_0603_1608Metric"
 			(at 48.26 33.02 0)
 			(hide yes)
@@
 			)
 		)
-		(property "Footprint" ""
+		(property "Footprint" "Capacitor_SMD:C_0603_1608Metric"
 			(at 47.625 53.975 0)
 			(hide yes)
@@
 			)
 		)
-		(property "Footprint" ""
+		(property "Footprint" "Resistor_SMD:R_0603_1608Metric"
 			(at 231.775 39.37 0)
 			(hide yes)
@@
 			)
 		)
-		(property "Value" "C_Small"
+		(property "Value" "100n"
 			(at 120.65 -25.4001 0)
-			(hide yes)
 			(show_name no)
 			(do_not_autoplace no)
@@
 			)
 		)
-		(property "Footprint" "Package_LCC:PLCC-44_16.6x16.6mm_P1.27mm"
+		(property "Footprint" "Capacitor_SMD:C_0603_1608Metric"
 			(at 118.11 -26.67 0)
 			(hide yes)
@@
 		(in_pos_files yes)
 		(dnp no)
-		(fields_autoplaced yes)
 		(property "Reference" "U7"
 			(at 221.8533 41.91 0)
@@
 			)
 		)
-		(property "Value" ""
-			(at 219.71 50.165 0)
+		(property "Value" "TLIN2021"
+			(at 226.695 59.69 0)
 			(show_name no)
 			(do_not_autoplace no)
@@
 			)
 		)
-		(property "Footprint" ""
+		(property "Footprint" "Package_SO:SOIC-8_5.3x5.3mm_P1.27mm"
 			(at 219.71 50.165 0)
 			(hide yes)
@@
 			)
 		)
-		(property "Datasheet" ""
+		(property "Datasheet" "https://www.ti.com/lit/ds/symlink/tlin2021-q1.pdf?ts=1791651585214&ref_url=https%253A%252F%252Fwww.ti.com%252Fproduct%252FTLIN2021-Q1"
 			(at 219.71 50.165 0)
 			(hide yes)
@@
 			)
 		)
-		(property "Footprint" ""
+		(property "Footprint" "Capacitor_SMD:C_0603_1608Metric"
 			(at 93.98 33.02 0)
 			(hide yes)
@@
 			)
 		)
-		(property "Footprint" ""
+		(property "Footprint" "Capacitor_SMD:C_0603_1608Metric"
 			(at 93.98 54.61 0)
 			(hide yes)
@@
 			)
 		)
-		(property "Footprint" ""
+		(property "Footprint" "Resistor_SMD:R_0603_1608Metric"
 			(at 251.46 46.99 0)
 			(hide yes)
@@
 		)
 	)
+	(group "58V Input Protection"
+		(lib_id "Library:58V Input Protection")
+		(members "039920a5-695e-4b0b-92a1-a9d93bb9aa40" "14a2bcd2-0b0b-417c-abef-b4772f598725"
+			"1a5dba01-d22e-4d50-ae97-f6c29ab4a3e8" "1ba5ba59-3fbc-46d1-ad23-22f7f940632b"
+			"227126fe-ec2a-403a-89f8-8c3685cfa63a" "24454cd8-48a6-416d-9d10-3f23077a96fa"
+			"546184cf-5025-4ff0-88f4-06033ec6feeb" "54d4a109-e532-447a-8b15-d39564f65bb4"
+			"6d4d7315-20c6-4e60-9c7b-6ed531273775" "70192817-541b-4d65-b888-ef1ed287b500"
+			"7640e62f-a2ea-4eab-b255-47a6b0d84539" "8bc74f71-4e48-4b37-8ce6-59cfe04cbb1a"
+			"907782af-2fae-44bf-b63f-95cd681c0815" "95870a02-f4a5-4db3-9b7f-c015508f90a0"
+			"bab0c6ef-a2a1-4f08-86ec-a664be821d88" "d272e794-b998-4d0e-9f71-a56010f7d280"
+			"e24fc70a-9455-45fa-9a8b-631bc2913d08" "e53b9037-b399-4ca5-b65a-b11e9ff315dd"
+			"e8215842-56c5-4bef-a41a-a677d545461d" "e82f08c6-bcce-40a8-a4f6-a779d973964d"
+			"fd1963e2-20b1-4168-80db-f104936f2179"
+		)
+	)

Commit message: 15-10-2026
Parts:
- removed C42, C43: 1n, Capacitor_SMD:C_0603_1608Metric, symbol Device:C_Small
- removed C46, C47, C48: 100n, Capacitor_SMD:C_0603_1608Metric, symbol Device:C_Small
- removed D10, D8: BAV99, Package_TO_SOT_SMD:SOT-23, symbol Diode:BAV99
- removed D11, D9: MM3Z62VB, Diode_SMD:D_SOD-323F, symbol Diode:MM3Zxx
- removed D14, D15: SMAJ58A, Diode_SMD:D_SMA, symbol Diode:SMAJ58A
- removed D19: BAS516, Diode_SMD:D_SOD-523, symbol Diode:BAS516
- removed E3, E4: SparkGap, Control_PCB:Sparkgap_2021-09-02, symbol Device:SparkGap
- removed Q10, Q11, Q4, Q7: BCX56, Package_TO_SOT_SMD:SOT-89-3, symbol Transistor_BJT:BCX56
- removed Q12, Q13, Q6, Q8: BC846, Package_TO_SOT_SMD:SOT-23, symbol Transistor_BJT:BC846
- removed Q9: PUMH11, Package_TO_SOT_SMD:SOT-363_SC-70-6, symbol Transistor_BJT:PUMX1
- removed R30, R31, R40, R42: 18k, Resistor_SMD:R_0603_1608Metric, symbol Device:R_Small
- removed R32, R44, R61: 100k, Resistor_SMD:R_0603_1608Metric, symbol Device:R_Small
- removed R33, R45: 4k7, Resistor_SMD:R_0603_1608Metric, symbol Device:R_Small
- removed R34, R36, R38, R39: 47, Resistor_SMD:R_0603_1608Metric, symbol Device:R_Small
- removed R35, R43, R62: 10k, Resistor_SMD:R_0603_1608Metric, symbol Device:R_Small
- removed R37, R41: 68k, Resistor_SMD:R_0603_1608Metric, symbol Device:R_Small
- removed R48, R49: 100, Resistor_SMD:R_1206_3216Metric, symbol Device:R_Small
- removed R56: 47k, Resistor_SMD:R_0603_1608Metric, symbol Device:R_Small
- removed TP10, TP11, TP12, TP13, TP18, TP23: TestPoint, TestPoint:TestPoint_Pad_D1.5mm, symbol Connector:TestPoint
- removed U7: TLIN2021, Package_SO:SOIC-8_5.3x5.3mm_P1.27mm, symbol Control_PCB:TLIN2021
Connections:
- net +12V is gone; now on net +5V: R71.2
- no-connect marks 2 -> 1
Other:
- note added: "Heartbeat"
- note removed: "Add Pull Down AND LIN Master Circuits!"
- note removed: "GPIO 3"
- moved on the sheet: C36, C37, C38, C39, C40, C41, C45, C53, D13, D16, D20, D4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

Commit message: Schematics mostly done
Parts:
- removed Q14: BCX56, Package_TO_SOT_SMD:SOT-89-3, symbol Transistor_BJT:BCX56
- added Q401: MMBT3904, Package_TO_SOT_SMD:SOT-23, symbol Transistor_BJT:MMBT3904
- R405: renamed from R69; value 1k -> 10k
- renumbered C44 to C401, C45 to C402, C53 to C403, C38 to C404, C37 to C405, C36 to C406, C40 to C407, C39 to C408, C41 to C409, D12 to D401, D13 to D402, D20 to D403, D4 to D404, D16 to D405, D6 to D406, E1 to E401, E2 to E402, E5 to E403, E6 to E404, L4 to L401, R71 to R401, R46 to R402, R47 to R403, R72 to R404, R70 to R406, R20 to R407, R21 to R408, R24 to R409, R25 to R410, R18 to R411, R19 to R412, R26 to R413, R27 to R414, R28 to R415, R29 to R416, TP6 to TP401, TP7 to TP402, TP4 to TP403, TP5 to TP404, TP8 to TP405, TP9 to TP406, U6 to U401
Connections:
- net GND: now also Q401.2 (E)
- net at R405.1, R406.2: now also Q401.1 (B)
- net at R401.1, R404.1: now also Q401.3 (C)

Commit message: Fixed some Schematic mistakes
- Fixed mirroers FETS
- Added voltage divider to TCAN INH
- fixed other minor mistakes
Parts:
- added C410: 47n, Capacitor_SMD:C_0603_1608Metric, symbol Device:C_Small
Connections:
- net AD_GPIO1: now also C410.1
- net GND: now also C410.2
Other:
- note added: "Place close to mcu pin"
Changed lines of the file:
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@@
+		)
+	)
+	(text "Place close\nto mcu pin\n"
+		(exclude_from_sim no)
+		(at 83.82 71.12 90)
+		(effects
+			(font
+				(size 1.27 1.27)
+			)
 		)
 	)
@@
 		(pts
 			(xy 134.62 92.71) (xy 135.89 92.71)
+		)
+		(stroke
+			(width 0)
+			(type default)
+		)
+	)
+	(wire
+		(pts
+			(xy 80.01 63.5) (xy 80.01 66.675)
 		)
 		(stroke
@@
 	)
 	(symbol
+		(lib_id "power:GND")
+		(at 80.01 71.755 0)
+		(unit 1)
+		(body_style 1)
+		(exclude_from_sim no)
+		(in_bom yes)
+		(on_board yes)
+		(in_pos_files yes)
+		(dnp no)
+		(fields_autoplaced yes)
+		(property "Reference" "#PWR0424"
+			(at 80.01 78.105 0)
+			(hide yes)
+			(show_name no)
+			(do_not_autoplace no)
+			(effects
+				(font
+					(size 1.27 1.27)
+				)
+			)
+		)
+		(property "Value" "GND"
+			(at 80.01 76.835 0)
+			(show_name no)
+			(do_not_autoplace no)
+			(effects
+				(font
+					(size 1.27 1.27)
+				)
+			)
+		)
+		(property "Footprint" ""
+			(at 80.01 71.755 0)
+			(hide yes)
+			(show_name no)
+			(do_not_autoplace no)
+			(effects
+				(font
+					(size 1.27 1.27)
+				)
+			)
+		)
+		(property "Datasheet" ""
+			(at 80.01 71.755 0)
+			(hide yes)
+			(show_name no)
+			(do_not_autoplace no)
+			(effects
+				(font
+					(size 1.27 1.27)
+				)
+			)
+		)
+		(property "Description" "Power symbol creates a global label with name \"GND\" , ground"
+			(at 80.01 71.755 0)
+			(hide yes)
+			(show_name no)
+			(do_not_autoplace no)
+			(effects
+				(font
+					(size 1.27 1.27)
+				)
+			)
+		)
+		(pin "1"
+		)
+		(instances
+			(project "Control_PCB"
+				(path "/dd8adfc1-6bab-46c3-a8c6-367c772462fc/e67d656d-c235-4d12-b9b1-11004966768e"
+					(reference "#PWR0424")
+					(unit 1)
+				)
+			)
+		)
+	)
+	(symbol
 		(lib_id "Device:C_Small")
 		(at 91.44 33.02 0)
@@
 					(unit 1)
 				)
+			)
+		)
+	)
+	(symbol
+		(lib_id "Device:C_Small")
+		(at 80.01 69.215 0)
+		(unit 1)
+		(body_style 1)
+		(exclude_from_sim no)
+		(in_bom yes)
+		(on_board yes)
+		(in_pos_files yes)
+		(dnp no)
+		(property "Reference" "C410"
+			(at 74.295 67.31 0)
+			(show_name no)
+			(do_not_autoplace no)
+			(effects
+				(font
+					(size 1.27 1.27)
+				)
+				(justify left)
+			)
+		)
+		(property "Value" "47n"
+			(at 75.565 71.12 0)
+			(show_name no)
+			(do_not_autoplace no)
+			(effects
+				(font
+					(size 1.27 1.27)
+				)
+				(justify left)
+			)
+		)
+		(property "Footprint" "Capacitor_SMD:C_0603_1608Metric"
+			(at 80.01 69.215 0)
+			(hide yes)
+			(show_name no)
+			(do_not_autoplace no)
+			(effects
+				(font
+					(size 1.27 1.27)
+				)
+			)
+		)
+		(property "Datasheet" ""
+			(at 80.01 69.215 0)
+			(hide yes)
+			(show_name no)
+			(do_not_autoplace no)
+			(effects
+				(font
+					(size 1.27 1.27)
+				)
+			)
+		)
+		(property "Description" "Unpolarized capacitor, small symbol"
+			(at 80.01 79.375 0)
+			(hide yes)
+			(show_name no)
+			(do_not_autoplace no)
+			(effects
+				(font
+					(size 1.27 1.27)
+				)
+			)
+		)
+		(pin "2"
+		)
+		(pin "1"
+		)
+		(instances
+			(project "Control_PCB"
+				(path "/dd8adfc1-6bab-46c3-a8c6-367c772462fc/e67d656d-c235-4d12-b9b1-11004966768e"
+					(reference "C410")
+					(unit 1)
+				)

Commit message: Surely i didnt miss anything else on the schematc...
Parts:
- added C411: 47n, Capacitor_SMD:C_0603_1608Metric, symbol Device:C_Small
- R401: value 100k -> 1k
- R404: value 100k -> 100
Connections:
- net AD_GPIO2: now also C411.1
- net GND: now also C411.2
Changed lines of the file:
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@@
 		)
 	)
+	(text "Place close\nto mcu pin\n"
+		(exclude_from_sim no)
+		(at 82.55 105.41 90)
+		(effects
+			(font
+				(size 1.27 1.27)
+			)
+		)
+	)
 	(text "INPUT 1"
 		(exclude_from_sim no)
@@
 	(wire
 		(pts
+			(xy 78.74 97.79) (xy 78.74 100.965)
+		)
+		(stroke
+			(width 0)
+			(type default)
+		)
+	)
+	(wire
+		(pts
 			(xy 200.66 100.33) (xy 200.66 101.6)
 		)
@@
 	)
 	(symbol
+		(lib_id "Device:C_Small")
+		(at 78.74 103.505 0)
+		(unit 1)
+		(body_style 1)
+		(exclude_from_sim no)
+		(in_bom yes)
+		(on_board yes)
+		(in_pos_files yes)
+		(dnp no)
+		(property "Reference" "C411"
+			(at 73.025 101.6 0)
+			(show_name no)
+			(do_not_autoplace no)
+			(effects
+				(font
+					(size 1.27 1.27)
+				)
+				(justify left)
+			)
+		)
+		(property "Value" "47n"
+			(at 74.295 105.41 0)
+			(show_name no)
+			(do_not_autoplace no)
+			(effects
+				(font
+					(size 1.27 1.27)
+				)
+				(justify left)
+			)
+		)
+		(property "Footprint" "Capacitor_SMD:C_0603_1608Metric"
+			(at 78.74 103.505 0)
+			(hide yes)
+			(show_name no)
+			(do_not_autoplace no)
+			(effects
+				(font
+					(size 1.27 1.27)
+				)
+			)
+		)
+		(property "Datasheet" ""
+			(at 78.74 103.505 0)
+			(hide yes)
+			(show_name no)
+			(do_not_autoplace no)
+			(effects
+				(font
+					(size 1.27 1.27)
+				)
+			)
+		)
+		(property "Description" "Unpolarized capacitor, small symbol"
+			(at 78.74 113.665 0)
+			(hide yes)
+			(show_name no)
+			(do_not_autoplace no)
+			(effects
+				(font
+					(size 1.27 1.27)
+				)
+			)
+		)
+		(pin "2"
+		)
+		(pin "1"
+		)
+		(instances
+			(project "Control_PCB"
+				(path "/dd8adfc1-6bab-46c3-a8c6-367c772462fc/e67d656d-c235-4d12-b9b1-11004966768e"
+					(reference "C411")
+					(unit 1)
+				)
+			)
+		)
+	)
+	(symbol
 		(lib_id "Device:R_Small")
 		(at 41.91 63.5 90)
@@
 		(dnp no)
 		(property "Reference" "R401"
-			(at 165.1 25.146 90)
+			(at 163.195 24.765 90)
 			(show_name no)
 			(do_not_autoplace no)
@@
 			)
 		)
-		(property "Value" "100k"
-			(at 166.878 24.892 90)
-			(hide yes)
+		(property "Value" "1k"
+			(at 167.005 26.035 90)
 			(show_name no)
 			(do_not_autoplace no)
@@
 		(dnp no)
 		(property "Reference" "R404"
-			(at 155.956 30.48 90)
+			(at 155.575 28.575 90)
 			(show_name no)
 			(do_not_autoplace no)
@@
 			)
 		)
-		(property "Value" "100k"
-			(at 155.702 28.702 90)
-			(hide yes)
+		(property "Value" "100"
+			(at 155.575 32.385 90)
 			(show_name no)
 			(do_not_autoplace no)
@@
 					(unit 1)
 				)
+			)
+		)
+	)
+	(symbol
+		(lib_id "power:GND")
+		(at 78.74 106.045 0)
+		(unit 1)
+		(body_style 1)
+		(exclude_from_sim no)
+		(in_bom yes)
+		(on_board yes)
+		(in_pos_files yes)
+		(dnp no)
+		(fields_autoplaced yes)
+		(property "Reference" "#PWR0425"
+			(at 78.74 112.395 0)
+			(hide yes)
+			(show_name no)
+			(do_not_autoplace no)
+			(effects
+				(font
+					(size 1.27 1.27)
+				)
+			)
+		)
+		(property "Value" "GND"
+			(at 78.74 111.125 0)
+			(show_name no)
+			(do_not_autoplace no)
+			(effects
+				(font
+					(size 1.27 1.27)
+				)
+			)
+		)
+		(property "Footprint" ""
+			(at 78.74 106.045 0)
+			(hide yes)
+			(show_name no)
+			(do_not_autoplace no)
+			(effects
+				(font
+					(size 1.27 1.27)
+				)
+			)
+		)
+		(property "Datasheet" ""
+			(at 78.74 106.045 0)
+			(hide yes)
+			(show_name no)
+			(do_not_autoplace no)
+			(effects
+				(font
+					(size 1.27 1.27)
+				)
+			)
+		)
+		(property "Description" "Power symbol creates a global label with name \"GND\" , ground"
+			(at 78.74 106.045 0)
+			(hide yes)
+			(show_name no)
+			(do_not_autoplace no)
+			(effects
+				(font
+					(size 1.27 1.27)
+				)
+			)
+		)
+		(pin "1"
+		)
+		(instances
+			(project "Control_PCB"
+				(path "/dd8adfc1-6bab-46c3-a8c6-367c772462fc/e67d656d-c235-4d12-b9b1-11004966768e"
+					(reference "#PWR0425")
+					(unit 1)
+				)
