File: Control_PCB/IO_Interface.kicad_sch (KiCad schematic)
At the start: 46 parts, among them Q401 MMBT3904, U401 TCAN1043xDxQ1

Commit message: 20/10-2026
Changed lines of the file:
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@@
 	)
 	(rectangle
-		(start -124.46 164.465)
-		(end -3.81 219.075)
+		(start 21.59 126.365)
+		(end 142.24 180.975)
 		(stroke
 			(width 0)
@@
 	(text "LIN"
 		(exclude_from_sim no)
-		(at -119.38 167.64 0)
+		(at 26.67 129.54 0)
 		(effects
 			(font
