File: Control_PCB/Power.kicad_sch (KiCad schematic)
At the start: 25 parts, among them U2 LM5164DDA, U3 TPS62A01APDDC

Commit message: 01-10-2026
Parts:
- removed C17: 100u, Package_SO:SOIC-8_3.9x4.9mm_P1.27mm, symbol Device:C_Polarized_Small
- added C17: 100u, Capacitor_SMD:C_1206_3216Metric, symbol Device:C_Small
- added C18, C19: 22u, Capacitor_SMD:C_0603_1608Metric, symbol Device:C_Small
- added C20, C21, C22, C23, C27: 1.5m, Capacitor_SMD:CP_Elec_8x10.5, symbol Device:C_Polarized_Small
- added C24, C25: 1u, Capacitor_SMD:C_0603_1608Metric, symbol Device:C_Small
- added C26: 100n, Capacitor_SMD:C_0603_1608Metric, symbol Device:C_Small
- added C28, C29: 2.2u, Capacitor_SMD:C_1206_3216Metric, symbol Device:C_Small
- added C30: 10u, Capacitor_SMD:C_0603_1608Metric, symbol Device:C_Small
- added D1: B360, Diode_SMD:D_SMB, symbol Diode:B360
- added D2: 1N5819WS, Diode_SMD:D_SOD-323, symbol Diode:1N5819WS
- added FB1: FerriteBead_Small, Inductor_SMD:L_0805_2012Metric, symbol Device:FerriteBead_Small
- added JP3: SolderJumper, Jumper:SolderJumper-2_P1.3mm_Bridged_Pad1.0x1.5mm, symbol Jumper:SolderJumper_2_Bridged
- added L3: 10u, Inductor_SMD:L_Bourns-SRN8040_8x8.15mm, symbol Device:L_Small
- added R10: 5.6, symbol Device:R_Small
- added R14: 0, Resistor_SMD:R_0603_1608Metric, symbol Device:R_Small
- added R15: 47k, Resistor_SMD:R_0603_1608Metric, symbol Device:R_Small
- added R16: 1, Resistor_SMD:R_1206_3216Metric, symbol Device:R_Small
- added U4: TLV61046ADB, Package_TO_SOT_SMD:SOT-23-6, symbol Regulator_Switching:TLV61046ADB
- added U5: (no value), Package_SO:SOP-4_7.5x4.1mm_P2.54mm, symbol Control_PCB:Photovoltaic
- C8: footprint Package_SO:SOIC-8_3.9x4.9mm_P1.27mm -> Capacitor_SMD:CP_Elec_8x10.5
Connections:
- net GND: now also C17.2, C18.2, C19.2, C20.2, C21.2, C22.2, C23.2, C24.2, C25.2, C26.2, C27.2, C28.2, C29.2, C30.2, U4.2 (GND)
- net PGOOD: now also R14.1
- net at L2.2, R8.1: now also JP2.1 (A), C18.1, C19.1
- net at C14.2, C15.1, C16.1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: now also C17.1
- net +5V: now reaches JP1.2 (B)
- net +5V: now also D1.2 (A), R16.1
- net +3V3: now reaches JP2.2 (B)
- net at U3.1 (EN), U3.4 (VIN): now also C24.1, D1.1 (K), D2.1 (K), R10.1
- new net: C20.1, C21.1, C22.1, C23.1, D2.2 (A), R10.2
- new net: C25.1, C26.1, C27.1, FB1.2, L3.1, R15.1, U4.3 (FB), U4.6 (VI)
- new net: L3.2, U4.1 (SW)
- new net: FB1.1, R16.2
- new net: C28.1, C29.1, R14.2, R15.2, U4.4 (EN)
- new net: C30.1, JP3.1 (A), U4.5 (VOUT)
- new net +12V: JP3.2 (B)
Other:
- note added: "12V - only for LIN...."
- note added: "3V3"
- note added: "Inrush Protection"
- note added: "Reverse Protection"
- note added: "What about just using USB..."
- moved on the sheet: C10, C11, C12, C13, C14, C15, C16, C8, C9, JP1, JP2, L1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

Commit message: 02-10-2026
Parts:
- added C31, C32: 270u, Capacitor_SMD:CP_Elec_8x10.5, symbol Device:C_Polarized_Small
- added C33, C34: 47u, Capacitor_SMD:CP_Elec_8x10.5, symbol Device:C_Polarized_Small
- added C35: 10n, Capacitor_SMD:C_0603_1608Metric, symbol Device:C_Small
- added D3: S3M-13-F, Diode_SMD:D_SOD-323, symbol Device:D
- added D5: SMDJ58CA, Diode_SMD:D_SMA, symbol Diode:SMAJ58CA
- added D7: MM5Z12V, Diode_SMD:D_SOD-523, symbol Diode:MM5Zxx
- added Q1: BC846, Package_TO_SOT_SMD:SOT-23, symbol Transistor_BJT:BC846
- added Q2, Q3: NTMFS016N06CT1G, Package_SO:ONSemi_SO-8FL_488AA, symbol Transistor_FET:NTMFS016N06CT1G
- added Q5: 2N7002, Package_TO_SOT_SMD:SOT-23, symbol Transistor_FET:2N7002
- added R11: 200, Resistor_SMD:R_0603_1608Metric, symbol Device:R_Small
- added R12: 10k, Resistor_SMD:R_0603_1608Metric, symbol Device:R_Small
- added R13: 1k, Resistor_SMD:R_0603_1608Metric, symbol Device:R_Small
- added R17: 47R - 3W, symbol Device:R
- added R22: 1Meg, Resistor_SMD:R_0603_1608Metric, symbol Device:R_Small
- added R23: 100k, Resistor_SMD:R_0603_1608Metric, symbol Device:R_Small
- added TP1, TP2, TP3: TestPoint, TestPoint:TestPoint_Pad_D1.5mm, symbol Connector:TestPoint
- U5: value (none) -> VOM1271T
Connections:
- net +3V3: now also U5.1
- net GND: now also C31.2, C32.2, C33.2, C34.2, D5.1 (A1), Q5.2 (S), R12.2, R23.1
- net at U5.2: now also R11.1
- net at U5.3: now also C35.2, D7.2 (A), Q2.1 (S), Q2.2 (S), Q2.3 (S), Q3.1 (S), Q3.2 (S), Q3.3 (S), TP3.1
- net at U5.4: now also C35.1, D7.1 (K), Q2.4 (G), Q3.4 (G), TP2.1
- new net: Q5.1 (G), R22.2, R23.2
- new net: Q1.1 (B), R12.1, R13.2
- new net: D3.1 (K), R17.1
- new net: Q1.2 (E), Q5.3 (D)
- new net: Q1.3 (C), R11.2
- new net ENA_INRUSH: R13.1
- new net VCC: C31.1, C32.1, C33.1, C34.1, Q3.5 (D), R17.2, TP1.1
- new net VCC_IN: D3.2 (A), D5.2 (A2), Q2.5 (D), R22.1
Other:
- note added: "+8V"
- note added: "Change the FETS to something rated for higher voltages!!! Also look at R_ON at 7V V_GS"
- note added: "Input Clamping"
- note added: "Inrush Protection Reverse Protection"
- note added: "≈ 17 mΩ @ 7V V_GS"
- note removed: "Inrush Protection"
- note removed: "Reverse Protection"
- moved on the sheet: C10, C11, C12, C13, C14, C15, C16, C17, C18, C19, C20, C21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

Commit message: 07-20-2026
Parts:
- added D17, D18: MM3Z56VB, Diode_SMD:D_SOD-323F, symbol Diode:MM3Zxx
- added R50, R53: 100k, symbol Device:R_Small
- added R51, R54, R57, R59: 220k, symbol Device:R_Small
- added R52, R55: 12k, symbol Device:R_Small
- added R58, R60: 68k, symbol Device:R_Small
- added TP14, TP15, TP16, TP17: TestPoint, TestPoint:TestPoint_Pad_D1.5mm, symbol Connector:TestPoint
Connections:
- net +12V: now also R57.1
- net +5V: now also R59.1
- net GND: now also D17.2 (A), D18.2 (A), R52.2, R55.2, R58.2, R60.2
- net VCC: now also R50.1
- net VCC_IN: now also R53.1
- new net: R50.2, R51.1
- new net: R53.2, R54.1
- new net AD_12V: R57.2, R58.1, TP16.1
- new net AD_5V: R59.2, R60.1, TP17.1
- new net AD_VCC: D17.1 (K), R51.2, R52.1, TP15.1
- new net AD_VCC_IN: D18.1 (K), R54.2, R55.1, TP14.1
Other:
- note added: "236.11mV/V"
- note added: "36.15mV/V"
- note added: "Voltage rate measurement"
- moved on the sheet: C25, C26, C27, C28, C29, C30, FB1, JP3, L3, R14, R15, R16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

Commit message: Before removing stuffs
Parts:
- removed C17: 100u, Capacitor_SMD:C_1206_3216Metric, symbol Device:C_Small
- removed C21, C22, C23, C27: 1.5m, Capacitor_SMD:CP_Elec_8x10.5, symbol Device:C_Polarized_Small
- removed C32: 270u, Capacitor_SMD:CP_Elec_8x10.5, symbol Device:C_Polarized_Small
- removed C33: 47u, Capacitor_SMD:CP_Elec_8x10.5, symbol Device:C_Polarized_Small
- added TP24: TestPoint, TestPoint:TestPoint_Pad_D1.5mm, symbol Connector:TestPoint
- C28, C29: footprint Capacitor_SMD:C_1206_3216Metric -> Capacitor_SMD:C_0805_2012Metric
- D17, D18: footprint Diode_SMD:D_SOD-323F -> Diode_SMD:D_SMA
- D5: footprint Diode_SMD:D_SMA -> Diode_SMD:D_SMB
- L3: footprint Inductor_SMD:L_Bourns-SRN8040_8x8.15mm -> Inductor_SMD:L_APV_ANR3012
- R10, R17: footprint (none) -> Resistor_SMD:R_2512_6332Metric
- R50, R51, R52, R53, R54, R55, R57, R58, R59, R60: footprint (none) -> Resistor_SMD:R_0603_1608Metric
Connections:
- net VCC: now also C10.1, C11.1, C8.1, C9.1, R1.1, U2.2 (VIN)
- net VCC_IN: now also TP24.1
- net at C12.1, U2.8 (SW): now also L1.1, R5.1
- net at C12.2, U2.7 (BST): no longer L1.1, R5.1
- net at R6.2, R7.1: now also C13.1, U2.5 (FB); no longer C13.2
- net at C14.1, R5.2: now also C13.2
Other:
- note added: "Remember To fix the Resistor values"
- moved on the sheet: C12, C13, C14, C20, C34, L1, R5

Commit message: 15-10-2026
Parts:
- removed C25: 1u, Capacitor_SMD:C_0603_1608Metric, symbol Device:C_Small
- removed C26: 100n, Capacitor_SMD:C_0603_1608Metric, symbol Device:C_Small
- removed C28, C29: 2.2u, Capacitor_SMD:C_0805_2012Metric, symbol Device:C_Small
- removed C30: 10u, Capacitor_SMD:C_0603_1608Metric, symbol Device:C_Small
- removed FB1: FerriteBead_Small, Inductor_SMD:L_0805_2012Metric, symbol Device:FerriteBead_Small
- removed JP3: SolderJumper, Jumper:SolderJumper-2_P1.3mm_Bridged_Pad1.0x1.5mm, symbol Jumper:SolderJumper_2_Bridged
- removed L3: 10u, Inductor_SMD:L_APV_ANR3012, symbol Device:L_Small
- removed R14: 0, Resistor_SMD:R_0603_1608Metric, symbol Device:R_Small
- removed R15: 47k, Resistor_SMD:R_0603_1608Metric, symbol Device:R_Small
- removed R16: 1, Resistor_SMD:R_1206_3216Metric, symbol Device:R_Small
- removed R57: 220k, Resistor_SMD:R_0603_1608Metric, symbol Device:R_Small
- removed R58: 68k, Resistor_SMD:R_0603_1608Metric, symbol Device:R_Small
- removed TP16: TestPoint, TestPoint:TestPoint_Pad_D1.5mm, symbol Connector:TestPoint
- removed U4: TLV61046ADB, Package_TO_SOT_SMD:SOT-23-6, symbol Regulator_Switching:TLV61046ADB
Other:
- note removed: "12V - only for LIN...."
- note removed: "What about just using USB..."
- moved on the sheet: C12, C13, C14, C20, C34, D18, JP1, L1, R5, R52, R53, R54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

Commit message: Schematics mostly done
Parts:
- removed C31: 270u, Capacitor_SMD:CP_Elec_8x10.5, symbol Device:C_Polarized_Small
- removed Q1: BC846, Package_TO_SOT_SMD:SOT-23, symbol Transistor_BJT:BC846
- removed Q2, Q3: NTMFS016N06CT1G, Package_SO:ONSemi_SO-8FL_488AA, symbol Transistor_FET:NTMFS016N06CT1G
- added C302, C303, C304: 47n, Capacitor_SMD:C_0603_1608Metric, symbol Device:C_Small
- added C305: 47u, Capacitor_SMD:CP_Elec_8x10.5, symbol Device:C_Polarized_Small
- added Q301: MMBT3904, Package_TO_SOT_SMD:SOT-23, symbol Transistor_BJT:MMBT3904
- added Q302, Q303: TPH4R50ANH1, Package_SON:Infineon_PG-TDSON-8_6.15x5.15mm, symbol Transistor_FET:NTMFS016N06CT1G
- C313: renamed from C16; value 10u -> 22u; footprint Capacitor_SMD:C_0603_1608Metric -> Capacitor_SMD:C_0805_2012Metric
- C316: renamed from C18; footprint Capacitor_SMD:C_0603_1608Metric -> Capacitor_SMD:C_0805_2012Metric
- C317: renamed from C19; footprint Capacitor_SMD:C_0603_1608Metric -> Capacitor_SMD:C_0805_2012Metric
- R304: renamed from R13; value 1k -> 10k
- R306: renamed from R12; value 10k -> 100k
- R316: renamed from R6; value 1k -> 390k
- R321: renamed from R7; value 1k -> 120k
- R324: renamed from R3; value 470k -> 240k
- renumbered C35 to C301, C34 to C306, C12 to C307, C8 to C308, C9 to C309, C10 to C310, C11 to C311, C15 to C312, C14 to C314, C24 to C315, C13 to C318, C20 to C319, D7 to D301, D5 to D302, D18 to D303, D17 to D304, D3 to D305, D1 to D306, D2 to D307, JP1 to JP301, JP2 to JP302, L1 to L301, L2 to L302, Q5 to Q304, R11 to R301, R53 to R302, R50 to R303, R54 to R305, R51 to R307, R59 to R308, R55 to R309, R52 to R310, R60 to R311, R22 to R312, R23 to R313, R17 to R314, R1 to R315, R5 to R317, R8 to R318, R10 to R319, R2 to R320, R9 to R322, R4 to R323, TP2 to TP301, TP14 to TP302, TP15 to TP303, TP17 to TP304, TP1 to TP305, TP3 to TP306, TP24 to TP307, U5 to U301, U3 to U302, U2 to U303
Connections:
- net AD_5V: now also C304.1
- net AD_VCC: now also C303.1; no longer D304.1 (K)
- net AD_VCC_IN: now also C302.1; no longer D303.1 (K)
- net GND: now also C302.2, C303.2, C304.2, C305.2
- net VCC: now also C305.1, Q303.1 (S), Q303.2 (S), Q303.3 (S)
- net VCC_IN: now also Q302.5 (D)
- net at C301.2, D301.2 (A), TP306.1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: now also Q302.1 (S), Q302.2 (S), Q302.3 (S), Q303.5 (D)
- net at C301.1, D301.1 (K), TP301.1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: now also Q302.4 (G), Q303.4 (G)
- net at R304.2, R306.1: now also Q301.1 (B)
- net at Q304.3 (D): now also Q301.2 (E)
- net at R303.2, R307.1: now also D304.1 (K)
- net at R301.2: now also Q301.3 (C)
- net at R302.2, R305.1: now also D303.1 (K)
Other:
- note added: "Place close to mcu pin"
- note removed: "CALCULATE HOW MUCH OUTPUT CAP I NEED I DONT LIKE C17..."
- note removed: "Change the FETS to something rated for higher voltages!!! Also look at R_ON at 7V V_GS"
- note removed: "Remember To fix the Resistor values"
- note removed: "≈ 17 mΩ @ 7V V_GS"
- moved on the sheet: D304, R302, R303, R307, R308, R310, R311, TP303, TP304

Commit message: Fixed some Schematic mistakes
- Fixed mirroers FETS
- Added voltage divider to TCAN INH
- fixed other minor mistakes
Parts:
- D302: footprint Diode_SMD:D_SMB -> Diode_SMD:D_SMC
- D303, D304: footprint Diode_SMD:D_SMA -> Diode_SMD:D_SOD-323F
- D305: footprint Diode_SMD:D_SOD-323 -> Diode_SMD:D_SMC
- D306: value B360 -> B360A; footprint Diode_SMD:D_SMB -> Diode_SMD:D_SMA
Connections:
- net VCC: now also Q303.5 (D); no longer Q303.1 (S), Q303.2 (S), Q303.3 (S)
- net at C301.2, D301.2 (A), Q302.1 (S)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: now also Q303.1 (S), Q303.2 (S), Q303.3 (S); no longer Q303.5 (D)
Other:
- moved on the sheet: Q303
Changed lines of the file:
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@@
 	(symbol
 		(lib_id "Transistor_FET:NTMFS016N06CT1G")
-		(at 120.65 57.15 90)
-		(mirror x)
+		(at 120.65 57.15 270)
 		(unit 1)
 		(body_style 1)
@@
 		(dnp no)
 		(property "Reference" "Q303"
-			(at 122.428 54.356 90)
+			(at 118.872 54.356 90)
 			(show_name no)
 			(do_not_autoplace no)
@@
 		)
 		(property "Value" "TPH4R50ANH1"
-			(at 120.015 62.865 90)
+			(at 121.285 62.865 90)
 			(show_name no)
 			(do_not_autoplace no)
@@
 		)
 		(property "Footprint" "Package_SON:Infineon_PG-TDSON-8_6.15x5.15mm"
-			(at 122.555 62.23 0)
+			(at 118.745 62.23 0)
 			(hide yes)
 			(show_name no)
@@
 		)
 		(property "Datasheet" "https://www.onsemi.cn/download/data-sheet/pdf/ntmfs015n10mcl-d.pdf"
-			(at 124.46 62.23 0)
+			(at 116.84 62.23 0)
 			(hide yes)
 			(show_name no)
@@
 			)
 		)
-		(property "Footprint" "Diode_SMD:D_SOD-323"
+		(property "Footprint" "Diode_SMD:D_SMC"
 			(at 99.06 73.66 0)
 			(hide yes)
@@
 			)
 		)
-		(property "Footprint" "Diode_SMD:D_SMA"
+		(property "Footprint" "Diode_SMD:D_SOD-323F"
 			(at 216.535 58.42 0)
 			(hide yes)
@@
 			)
 		)
-		(property "Footprint" "Diode_SMD:D_SMA"
+		(property "Footprint" "Diode_SMD:D_SOD-323F"
 			(at 179.705 57.15 0)
 			(hide yes)
@@
 			)
 		)
-		(property "Value" "B360"
+		(property "Value" "B360A"
 			(at 193.04 94.2974 90)
 			(show_name no)
@@
 			)
 		)
-		(property "Footprint" "Diode_SMD:D_SMB"
+		(property "Footprint" "Diode_SMD:D_SMA"
 			(at 194.945 92.71 0)
 			(hide yes)
@@
 			)
 		)
-		(property "Footprint" "Diode_SMD:D_SMB"
+		(property "Footprint" "Diode_SMD:D_SMC"
 			(at 34.29 48.26 0)
 			(hide yes)

Commit message: Updated schematic started on layout for motor PCB
Parts:
- removed C306: 47u, Capacitor_SMD:CP_Elec_8x10.5, symbol Device:C_Polarized_Small
Changed lines of the file:
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@@
 	)
 	(junction
-		(at 140.97 59.69)
-		(diameter 0)
-		(color 0 0 0 0)
-	)
-	(junction
 		(at 214.63 96.52)
 		(diameter 0)
@@
 	)
 	(junction
-		(at 137.16 71.12)
-		(diameter 0)
-		(color 0 0 0 0)
-	)
-	(junction
 		(at 231.14 54.61)
 		(diameter 0)
@@
 	(wire
 		(pts
-			(xy 133.35 71.12) (xy 137.16 71.12)
-		)
-		(stroke
-			(width 0)
-			(type default)
-		)
-	)
-	(wire
-		(pts
 			(xy 232.41 96.52) (xy 236.22 96.52)
 		)
@@
 	(wire
 		(pts
-			(xy 137.16 71.12) (xy 140.97 71.12)
-		)
-		(stroke
-			(width 0)
-			(type default)
-		)
-	)
-	(wire
-		(pts
 			(xy 105.41 36.83) (xy 106.68 36.83)
 		)
@@
 	(wire
 		(pts
-			(xy 140.97 59.69) (xy 154.94 59.69)
-		)
-		(stroke
-			(width 0)
-			(type default)
-		)
-	)
-	(wire
-		(pts
 			(xy 102.87 73.66) (xy 111.76 73.66)
 		)
@@
 	(wire
 		(pts
-			(xy 140.97 68.58) (xy 140.97 71.12)
-		)
-		(stroke
-			(width 0)
-			(type default)
-		)
-	)
-	(wire
-		(pts
-			(xy 133.35 68.58) (xy 133.35 71.12)
+			(xy 133.35 68.58) (xy 133.35 71.755)
 		)
 		(stroke
@@
 	(wire
 		(pts
-			(xy 133.35 59.69) (xy 140.97 59.69)
+			(xy 133.35 59.69) (xy 154.94 59.69)
 		)
 		(stroke
@@
 	(wire
 		(pts
-			(xy 137.16 71.12) (xy 137.16 72.39)
-		)
-		(stroke
-			(width 0)
-			(type default)
-		)
-	)
-	(wire
-		(pts
 			(xy 256.54 45.72) (xy 256.54 46.99)
 		)
@@
 	(wire
 		(pts
-			(xy 140.97 59.69) (xy 140.97 63.5)
-		)
-		(stroke
-			(width 0)
-			(type default)
-		)
-	)
-	(wire
-		(pts
 			(xy 106.68 27.94) (xy 106.68 29.21)
 		)
@@
 	(symbol
 		(lib_id "power:GND")
-		(at 137.16 72.39 0)
+		(at 133.35 71.755 0)
 		(unit 1)
 		(body_style 1)
@@
 		(dnp no)
 		(property "Reference" "#PWR0316"
-			(at 137.16 78.74 0)
+			(at 133.35 78.105 0)
 			(hide yes)
 			(show_name no)
@@
 		)
 		(property "Value" "GND"
-			(at 137.16 76.2 0)
+			(at 133.35 75.565 0)
 			(show_name no)
 			(do_not_autoplace no)
@@
 		)
 		(property "Footprint" ""
-			(at 137.16 72.39 0)
+			(at 133.35 71.755 0)
 			(hide yes)
 			(show_name no)
@@
 		)
 		(property "Datasheet" ""
-			(at 137.16 72.39 0)
+			(at 133.35 71.755 0)
 			(hide yes)
 			(show_name no)
@@
 		)
 		(property "Description" "Power symbol creates a global label with name \"GND\" , ground"
-			(at 137.16 72.39 0)
+			(at 133.35 71.755 0)
 			(hide yes)
 			(show_name no)
@@
 					(unit 1)
 				)
-			)
-		)
-	)
-	(symbol
-		(lib_id "Device:C_Polarized_Small")
-		(at 140.97 66.04 0)
-		(unit 1)
-		(body_style 1)
-		(exclude_from_sim no)
-		(in_bom yes)
-		(on_board yes)
-		(in_pos_files yes)
-		(dnp no)
-		(property "Reference" "C306"
-			(at 141.478 64.262 0)
-			(show_name no)
-			(do_not_autoplace no)
-			(effects
-				(font
-					(size 1.27 1.27)
-				)
-				(justify left)
-			)
-		)
-		(property "Value" "47u"
-			(at 141.224 68.072 0)
-			(show_name no)
-			(do_not_autoplace no)
-			(effects
-				(font
-					(size 1.27 1.27)
-				)
-				(justify left)
-			)
-		)
-		(property "Footprint" "Capacitor_SMD:CP_Elec_8x10.5"
-			(at 140.97 66.04 0)
-			(hide yes)
-			(show_name no)
-			(do_not_autoplace no)
-			(effects
-				(font
-					(size 1.27 1.27)
-				)
-			)
-		)
-		(property "Datasheet" "https://jlcpcb.com/partdetail/ROQANG-SVC2A470M0810/C49253409"
-			(at 140.97 66.04 0)
-			(hide yes)
-			(show_name no)
-			(do_not_autoplace no)
-			(effects
-				(font
-					(size 1.27 1.27)
-				)
-			)
-		)
-		(property "Description" "100V"
-			(at 143.51 69.85 0)
-			(show_name no)
-			(do_not_autoplace no)
-			(effects
-				(font
-					(size 1.27 1.27)
-				)
-			)
-		)
-		(pin "1"
-		)
-		(pin "2"
-		)
-		(instances
-			(project "Control_PCB"
-				(path "/dd8adfc1-6bab-46c3-a8c6-367c772462fc/5f352cea-9e1c-4ca2-9247-1e9fdcf12f9b"
-					(reference "C306")
-					(unit 1)
-				)
