File: Control_PCB/Power.kicad_sch (KiCad schematic)
At the start: 67 parts, among them Q301 MMBT3904, Q302 TPH4R50ANH1, Q303 TPH4R50ANH1, Q304 2N7002, U301 VOM1271T, U302 TPS62A01APDDC, U303 LM5164DDA

Commit message: 20/10-2026
Parts:
- U301: footprint Package_SO:SOP-4_7.5x4.1mm_P2.54mm -> Control_PCB:SOP-4_VIS
Changed lines of the file:
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@@
 			)
 		)
-		(property "Footprint" "Package_SO:SOP-4_7.5x4.1mm_P2.54mm"
+		(property "Footprint" "Control_PCB:SOP-4_VIS"
 			(at 90.17 26.67 0)
 			(hide yes)
