File: Control_PCB/Control_PCB.kicad_pcb (KiCad board)
At the start: 2 copper layers, 33 parts, among them U1 STM32G473VET3, U2 LM5164DDA, U3 TPS62A01APDDC

Commit message: 01-10-2026
Parts:
- added C18: 22u, Capacitor_SMD:C_0603_1608Metric, F.Cu at (52.0, 47.8)
- added C19: 22u, Capacitor_SMD:C_0603_1608Metric, F.Cu at (53.5, 56.3)
- added C20: 1.5m, Capacitor_SMD:CP_Elec_8x10.5, F.Cu at (62.0, 27.5)
- added C21: 1.5m, Capacitor_SMD:CP_Elec_8x10.5, F.Cu at (61.8, 38.5)
- added C22: 1.5m, Capacitor_SMD:CP_Elec_8x10.5, F.Cu at (62.8, 49.5)
- added C23: 1.5m, Capacitor_SMD:CP_Elec_8x10.5, F.Cu at (62.5, 60.5)
- added C24: 1u, Capacitor_SMD:C_0603_1608Metric, F.Cu at (78.8, 37.1)
- added D1: B360, Diode_SMD:D_SMB, F.Cu at (78.0, 32.0)
- added D2: 1N5819WS, Diode_SMD:D_SOD-323, F.Cu at (74.7, 37.4)
- C17: footprint Package_SO:SOIC-8_3.9x4.9mm_P1.27mm -> Capacitor_SMD:C_1206_3216Metric
- C8: footprint Package_SO:SOIC-8_3.9x4.9mm_P1.27mm -> Capacitor_SMD:CP_Elec_8x10.5
- moved C8 4.61 mm to (104.0, 42.0)
- moved C17 3.91 mm to (90.0, 42.5)
Connections:
- JP1 pad 2: unconnected-(JP1-B-Pad2) -> +5V
- JP2 pad 1: unconnected-(JP2-A-Pad1) -> Net-(JP2-A)
- JP2 pad 2: unconnected-(JP2-B-Pad2) -> +3V3
- L2 pad 2: Net-(L2-Pad2) -> Net-(JP2-A)
- R8 pad 1: Net-(L2-Pad2) -> Net-(JP2-A)

Commit message: 02-10-2026
Parts:
- added C25: 1u, Capacitor_SMD:C_0603_1608Metric, F.Cu at (48.9, 72.3)
- added C26: 100n, Capacitor_SMD:C_0603_1608Metric, F.Cu at (48.9, 74.8)
- added C27: 1.5m, Capacitor_SMD:CP_Elec_8x10.5, F.Cu at (40.2, 76.0)
- added C28: 2.2u, Capacitor_SMD:C_1206_3216Metric, F.Cu at (54.6, 108.6)
- added C29: 2.2u, Capacitor_SMD:C_1206_3216Metric, F.Cu at (54.6, 111.9)
- added C30: 10u, Capacitor_SMD:C_0603_1608Metric, F.Cu at (48.9, 77.3)
- added C31: 270u, Capacitor_SMD:CP_Elec_8x10.5, F.Cu at (40.2, 86.1)
- added C32: 270u, Capacitor_SMD:CP_Elec_8x10.5, F.Cu at (40.2, 96.1)
- added C33: 47u, Capacitor_SMD:CP_Elec_8x10.5, F.Cu at (40.2, 106.2)
- added C34: 47u, Capacitor_SMD:CP_Elec_8x10.5, F.Cu at (40.2, 116.2)
- added C35: 10n, Capacitor_SMD:C_0603_1608Metric, F.Cu at (48.9, 79.8)
- added C36: 100n, Capacitor_SMD:C_0603_1608Metric, F.Cu at (66.9, 72.3)
- added C37: 100n, Capacitor_SMD:C_0603_1608Metric, F.Cu at (66.9, 74.8)
- added C38: 100n, Capacitor_SMD:C_0603_1608Metric, F.Cu at (66.9, 77.3)
- added C39: 4.7n, Capacitor_SMD:C_0603_1608Metric, F.Cu at (66.9, 79.8)
- added D3: S3M-13-F, Diode_SMD:D_SOD-323, F.Cu at (59.6, 108.4)
- added D5: SMDJ58CA, Diode_SMD:D_SMA, F.Cu at (55.8, 104.6)
- added D7: MM5Z12V, Diode_SMD:D_SOD-523, F.Cu at (59.2, 111.1)
- added FB1: FerriteBead_Small, Inductor_SMD:L_0805_2012Metric, F.Cu at (59.6, 119.6)
- added JP3: SolderJumper, Jumper:SolderJumper-2_P1.3mm_Bridged_Pad1.0x1.5mm, F.Cu at (53.9, 118.7)
- added L3: 10u, Inductor_SMD:L_Bourns-SRN8040_8x8.15mm, F.Cu at (55.3, 96.6)
- added Q1: BC846, Package_TO_SOT_SMD:SOT-23, F.Cu at (49.3, 104.6)
- added Q2: NTMFS016N06CT1G, Package_SO:ONSemi_SO-8FL_488AA, F.Cu at (58.9, 74.6)
- added Q3: NTMFS016N06CT1G, Package_SO:ONSemi_SO-8FL_488AA, F.Cu at (58.9, 81.7)
- added Q5: 2N7002, Package_TO_SOT_SMD:SOT-23, F.Cu at (49.3, 109.0)
- added R11: 200, Resistor_SMD:R_0603_1608Metric, F.Cu at (48.9, 82.3)
- added R12: 10k, Resistor_SMD:R_0603_1608Metric, F.Cu at (48.9, 84.8)
- added R13: 1k, Resistor_SMD:R_0603_1608Metric, F.Cu at (52.9, 72.3)
- added R14: 0, Resistor_SMD:R_0603_1608Metric, F.Cu at (52.9, 74.8)
- added R15: 47k, Resistor_SMD:R_0603_1608Metric, F.Cu at (52.9, 77.3)
- added R16: 1, Resistor_SMD:R_1206_3216Metric, F.Cu at (54.6, 115.3)
- added R18: 60, Resistor_SMD:R_0603_1608Metric, F.Cu at (66.9, 82.3)
- added R19: 60, Resistor_SMD:R_0603_1608Metric, F.Cu at (66.9, 84.8)
- added R22: 1Meg, Resistor_SMD:R_0603_1608Metric, F.Cu at (52.9, 79.8)
- added R23: 100k, Resistor_SMD:R_0603_1608Metric, F.Cu at (52.9, 82.3)
- added TP1: TestPoint, TestPoint:TestPoint_Pad_D1.5mm, F.Cu at (48.6, 93.5)
- added TP2: TestPoint, TestPoint:TestPoint_Pad_D1.5mm, F.Cu at (48.6, 97.0)
- added TP3: TestPoint, TestPoint:TestPoint_Pad_D1.5mm, F.Cu at (48.6, 100.6)
- added TP4: TestPoint, TestPoint:TestPoint_Pad_D1.5mm, F.Cu at (79.2, 72.8)
- added TP5: TestPoint, TestPoint:TestPoint_Pad_D1.5mm, F.Cu at (79.2, 76.3)
- added U4: TLV61046ADB, Package_TO_SOT_SMD:SOT-23-6, F.Cu at (59.9, 116.0)
- added U5: VOM1271T, Package_SO:SOP-4_7.5x4.1mm_P2.54mm, F.Cu at (53.2, 88.9)
- added U6: TCAN1043xDxQ1, Package_SO:SOIC-14_3.9x8.7mm_P1.27mm, F.Cu at (73.2, 76.3)
Connections:
- U1 pad 61: unconnected-(U1A-PD14-Pad61) -> /mcu/CAN_STB
- U1 pad 9: unconnected-(U1A-PC15-OSC32_OUT-Pad9) -> /mcu/CAN_FAULT
- U1 pad 96: unconnected-(U1A-PB9-Pad96) -> /mcu/CAN_ENA

Commit message: 07-20-2026
Parts:
- added C40: 1n, Capacitor_SMD:C_0603_1608Metric, F.Cu at (105.6, 39.2)
- added C41: 1n, Capacitor_SMD:C_0603_1608Metric, F.Cu at (105.6, 41.7)
- added C42: 1n, Capacitor_SMD:C_0603_1608Metric, F.Cu at (105.6, 44.2)
- added C43: 1n, Capacitor_SMD:C_0603_1608Metric, F.Cu at (105.6, 46.7)
- added D10: BAV99, Package_TO_SOT_SMD:SOT-23, F.Cu at (95.0, 34.6)
- added D11: MM3Z62VB, Diode_SMD:D_SOD-323F, F.Cu at (111.3, 60.8)
- added D12: SMAJ58A, Diode_SMD:D_SMA, F.Cu at (133.6, 29.5)
- added D13: SMAJ58A, Diode_SMD:D_SMA, F.Cu at (133.6, 34.0)
- added D14: SMAJ58A, Diode_SMD:D_SMA, F.Cu at (133.6, 38.6)
- added D15: SMAJ58A, Diode_SMD:D_SMA, F.Cu at (133.6, 43.1)
- added D4: MM3Z62VB, Diode_SMD:D_SOD-323F, F.Cu at (111.3, 52.0)
- added D6: MM3Z62VB, Diode_SMD:D_SOD-323F, F.Cu at (111.3, 54.9)
- added D8: BAV99, Package_TO_SOT_SMD:SOT-23, F.Cu at (95.0, 30.1)
- added D9: MM3Z62VB, Diode_SMD:D_SOD-323F, F.Cu at (111.3, 57.9)
- added E1: SparkGap, Control_PCB:Sparkgap_2021-09-02, F.Cu at (128.0, 29.2)
- added E2: SparkGap, Control_PCB:Sparkgap_2021-09-02, F.Cu at (128.0, 31.8)
- added E3: SparkGap, Control_PCB:Sparkgap_2021-09-02, F.Cu at (128.0, 34.4)
- added E4: SparkGap, Control_PCB:Sparkgap_2021-09-02, F.Cu at (128.0, 37.0)
- added E5: SparkGap, Control_PCB:Sparkgap_2021-09-02, F.Cu at (128.0, 39.6)
- added E6: SparkGap, Control_PCB:Sparkgap_2021-09-02, F.Cu at (128.0, 42.2)
- added L4: DR331-513AE, Inductor_SMD:L_CommonMode_Bourns_DR331, F.Cu at (157.4, 33.6)
- added Q10: BCX56, Package_TO_SOT_SMD:SOT-89-3, F.Cu at (100.8, 43.2)
- added Q11: BCX56, Package_TO_SOT_SMD:SOT-89-3, F.Cu at (100.8, 49.4)
- added Q12: BC846, Package_TO_SOT_SMD:SOT-23, F.Cu at (95.0, 47.9)
- added Q13: BC846, Package_TO_SOT_SMD:SOT-23, F.Cu at (95.0, 52.4)
- added Q4: BCX56, Package_TO_SOT_SMD:SOT-89-3, F.Cu at (100.8, 31.0)
- added Q6: BC846, Package_TO_SOT_SMD:SOT-23, F.Cu at (95.0, 39.0)
- added Q7: BCX56, Package_TO_SOT_SMD:SOT-89-3, F.Cu at (100.8, 37.1)
- added Q8: BC846, Package_TO_SOT_SMD:SOT-23, F.Cu at (95.0, 43.5)
- added Q9: PUMH11, Package_TO_SOT_SMD:SOT-363_SC-70-6, F.Cu at (123.9, 52.3)
- added R20: 18k, Resistor_SMD:R_0603_1608Metric, F.Cu at (109.6, 31.7)
- added R21: 18k, Resistor_SMD:R_0603_1608Metric, F.Cu at (109.6, 34.2)
- added R24: 100k, Resistor_SMD:R_0603_1608Metric, F.Cu at (109.6, 36.7)
- added R25: 4k7, Resistor_SMD:R_0603_1608Metric, F.Cu at (109.6, 39.2)
- added R26: 18k, Resistor_SMD:R_0603_1608Metric, F.Cu at (109.6, 41.7)
- added R27: 18k, Resistor_SMD:R_0603_1608Metric, F.Cu at (109.6, 44.2)
- added R28: 100k, Resistor_SMD:R_0603_1608Metric, F.Cu at (109.6, 46.7)
- added R29: 4k7, Resistor_SMD:R_0603_1608Metric, F.Cu at (109.6, 49.2)
- added R30: 18k, Resistor_SMD:R_0603_1608Metric, F.Cu at (113.6, 29.2)
- added R31: 18k, Resistor_SMD:R_0603_1608Metric, F.Cu at (113.6, 31.7)
- added R32: 100k, Resistor_SMD:R_0603_1608Metric, F.Cu at (113.6, 34.2)
- added R33: 4k7, Resistor_SMD:R_0603_1608Metric, F.Cu at (113.6, 36.7)
- added R34: 47, Resistor_SMD:R_0603_1608Metric, F.Cu at (113.6, 39.2)
- added R35: 10k, Resistor_SMD:R_0603_1608Metric, F.Cu at (113.6, 41.7)
- added R36: 47, Resistor_SMD:R_0603_1608Metric, F.Cu at (113.6, 44.2)
- added R37: 68k, Resistor_SMD:R_0603_1608Metric, F.Cu at (113.6, 46.7)
- added R38: 47, Resistor_SMD:R_0603_1608Metric, F.Cu at (113.6, 49.2)
- added R39: 47, Resistor_SMD:R_0603_1608Metric, F.Cu at (117.6, 29.2)
- added R40: 18k, Resistor_SMD:R_0603_1608Metric, F.Cu at (117.6, 31.7)
- added R41: 68k, Resistor_SMD:R_0603_1608Metric, F.Cu at (117.6, 34.2)
- added R42: 18k, Resistor_SMD:R_0603_1608Metric, F.Cu at (117.6, 36.7)
- added R43: 10k, Resistor_SMD:R_0603_1608Metric, F.Cu at (117.6, 39.2)
- added R44: 100k, Resistor_SMD:R_0603_1608Metric, F.Cu at (117.6, 41.7)
- added R45: 4k7, Resistor_SMD:R_0603_1608Metric, F.Cu at (117.6, 44.2)
- added R46: 100, Resistor_SMD:R_1206_3216Metric, F.Cu at (106.4, 52.1)
- added R47: 100, Resistor_SMD:R_1206_3216Metric, F.Cu at (106.4, 55.5)
- added R48: 100, Resistor_SMD:R_1206_3216Metric, F.Cu at (106.4, 58.8)
- added R49: 100, Resistor_SMD:R_1206_3216Metric, F.Cu at (106.4, 62.1)
- added TP10: TestPoint, TestPoint:TestPoint_Pad_D1.5mm, F.Cu at (124.9, 33.2)
- added TP11: TestPoint, TestPoint:TestPoint_Pad_D1.5mm, F.Cu at (124.9, 36.8)
- added TP12: TestPoint, TestPoint:TestPoint_Pad_D1.5mm, F.Cu at (124.9, 40.3)
- added TP13: TestPoint, TestPoint:TestPoint_Pad_D1.5mm, F.Cu at (124.9, 43.9)
- added TP6: TestPoint, TestPoint:TestPoint_Pad_D1.5mm, F.Cu at (121.4, 36.8)
- added TP7: TestPoint, TestPoint:TestPoint_Pad_D1.5mm, F.Cu at (121.4, 40.3)
- added TP8: TestPoint, TestPoint:TestPoint_Pad_D1.5mm, F.Cu at (121.4, 43.9)
- added TP9: TestPoint, TestPoint:TestPoint_Pad_D1.5mm, F.Cu at (124.9, 29.7)
- moved Q1 80.4 mm to (79.6, 30.1)
- moved Q5 80.4 mm to (79.6, 34.6)
- moved C11 75.5 mm to (53.1, 79.7)
- moved D3 72.8 mm to (87.7, 41.2)
- moved R19 70.1 mm to (109.6, 29.2)
- moved C13 66.9 mm to (60.3, 79.1)
- moved D5 65.2 mm to (81.2, 44.6)
- moved TP4 60.3 mm to (121.4, 29.7)
- moved TP5 60.3 mm to (121.4, 33.2)
- moved C29 58.7 mm to (86.3, 62.5)
- moved C28 58.7 mm to (86.3, 59.1)
- moved C38 57.9 mm to (105.6, 34.2)
- moved C36 57.9 mm to (105.6, 29.2)
- moved C37 57.9 mm to (105.6, 31.7)
- moved C39 57.9 mm to (105.6, 36.7)
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Connections:
- net /IO_Interface/CANH renamed Net-(U6-CANH)
- net /IO_Interface/CANL renamed Net-(U6-CANL)

Commit message: Before removing stuffs
Parts:
- removed C17: 100u, Capacitor_SMD:C_1206_3216Metric
- removed C21, C22, C23, C27: 1.5m, Capacitor_SMD:CP_Elec_8x10.5
- removed C32: 270u, Capacitor_SMD:CP_Elec_8x10.5
- removed C33: 47u, Capacitor_SMD:CP_Elec_8x10.5
- added C44: 100n, Capacitor_SMD:C_0603_1608Metric, F.Cu at (219.1, 62.0)
- added C45: 100n, Capacitor_SMD:C_0603_1608Metric, F.Cu at (223.3, 62.0)
- added C46: 100n, Capacitor_SMD:C_0603_1608Metric, F.Cu at (227.6, 62.0)
- added C47: 100n, Capacitor_SMD:C_0603_1608Metric, F.Cu at (231.9, 62.0)
- added C48: 100n, Capacitor_SMD:C_0603_1608Metric, F.Cu at (282.5, -25.2)
- added C49: 24p, Capacitor_SMD:C_0603_1608Metric, F.Cu at (205.3, 131.8)
- added C50: 24p, Capacitor_SMD:C_0603_1608Metric, F.Cu at (205.3, 134.9)
- added C51: 1u, Capacitor_SMD:C_0603_1608Metric, F.Cu at (216.1, 119.7)
- added C52: 10n, Capacitor_SMD:C_0603_1608Metric, F.Cu at (199.2, 140.9)
- added C53: 100n, Capacitor_SMD:C_0603_1608Metric, F.Cu at (258.4, 145.1)
- added D16: ESD2CANFD60-Q1, Package_TO_SOT_SMD:SOT-23-3, F.Cu at (260.8, 149.4)
- added D17: MM3Z56VB, Diode_SMD:D_SMA, F.Cu at (55.2, 123.8)
- added D18: MM3Z56VB, Diode_SMD:D_SMA, F.Cu at (55.5, 131.7)
- added D19: BAS516, Diode_SMD:D_SOD-523, F.Cu at (289.1, -11.2)
- added D20: SMAJ16A, Diode_SMD:D_SMA, F.Cu at (261.1, 143.8)
- added D21: PESD5V2S2UT, Package_TO_SOT_SMD:SOT-23, F.Cu at (133.1, 47.7)
- added J1: Minifit 2x3, Connector_Molex:Molex_Mini-Fit_Jr_5569-06A2_2x03_P4.20mm_Horizontal, F.Cu at (176.6, 45.1)
- added J2: Conn_01x09, Control_PCB:Molex_Micro-Fit_3x03_P3.00mm, F.Cu at (228.3, 38.2)
- added J3: Conn_01x05, Control_PCB:1411976, F.Cu at (269.6, 148.1)
- added J4: Micro Match, Control_PCB:CONN6_7-188275-6_TEC, F.Cu at (159.8, 145.9)
- added Q14: BCX56, Package_TO_SOT_SMD:SOT-89-3, F.Cu at (268.8, 128.6)
- added R10: 5.6, Resistor_SMD:R_2512_6332Metric, F.Cu at (88.1, -84.3)
- added R17: 47R - 3W, Resistor_SMD:R_2512_6332Metric, F.Cu at (194.9, 70.6)
- added R50: 100k, Resistor_SMD:R_0603_1608Metric, F.Cu at (53.2, 109.6)
- added R51: 220k, Resistor_SMD:R_0603_1608Metric, F.Cu at (53.2, 112.1)
- added R52: 12k, Resistor_SMD:R_0603_1608Metric, F.Cu at (53.2, 114.6)
- added R53: 100k, Resistor_SMD:R_0603_1608Metric, F.Cu at (53.2, 117.2)
- added R54: 220k, Resistor_SMD:R_0603_1608Metric, F.Cu at (53.2, 119.7)
- added R55: 12k, Resistor_SMD:R_0603_1608Metric, F.Cu at (57.2, 109.6)
- added R56: 47k, Resistor_SMD:R_0603_1608Metric, F.Cu at (296.4, -15.6)
- added R57: 220k, Resistor_SMD:R_0603_1608Metric, F.Cu at (57.2, 112.1)
- added R58: 68k, Resistor_SMD:R_0603_1608Metric, F.Cu at (57.2, 114.6)
- added R59: 220k, Resistor_SMD:R_0603_1608Metric, F.Cu at (57.2, 117.2)
- added R60: 68k, Resistor_SMD:R_0603_1608Metric, F.Cu at (57.2, 119.7)
- added R61: 100k, Resistor_SMD:R_0603_1608Metric, F.Cu at (296.4, -13.1)
- added R62: 10k, Resistor_SMD:R_0603_1608Metric, F.Cu at (296.4, -10.6)
- added R63: 100, Resistor_SMD:R_0603_1608Metric, F.Cu at (131.9, 43.8)
- added R64: 100, Resistor_SMD:R_0603_1608Metric, F.Cu at (134.2, 43.8)
- added R65: 470k, Resistor_SMD:R_0603_1608Metric, F.Cu at (229.6, 130.2)
- added R66: 15k, Resistor_SMD:R_0603_1608Metric, F.Cu at (216.1, 117.9)
- added R67: 100k, Resistor_SMD:R_0603_1608Metric, F.Cu at (216.1, 121.4)
- added R68: 10k, Resistor_SMD:R_0603_1608Metric, F.Cu at (63.2, 119.7)
- added R69: 1k, Resistor_SMD:R_0603_1608Metric, F.Cu at (262.0, 126.8)
- added R70: 100k, Resistor_SMD:R_0603_1608Metric, F.Cu at (264.6, 126.0)
- added R71: 100k, Resistor_SMD:R_0603_1608Metric, F.Cu at (264.6, 129.3)
- added R72: 100k, Resistor_SMD:R_0603_1608Metric, F.Cu at (262.0, 128.6)
- added TP14: TestPoint, TestPoint:TestPoint_Pad_D1.5mm, F.Cu at (53.6, 136.5)
- added TP15: TestPoint, TestPoint:TestPoint_Pad_D1.5mm, F.Cu at (57.2, 136.6)
- added TP16: TestPoint, TestPoint:TestPoint_Pad_D1.5mm, F.Cu at (60.8, 136.6)
- added TP17: TestPoint, TestPoint:TestPoint_Pad_D1.5mm, F.Cu at (64.3, 136.6)
- added TP18: TestPoint, TestPoint:TestPoint_Pad_D1.5mm, F.Cu at (279.3, -15.1)
- added TP19: TestPoint, TestPoint:TestPoint_Pad_D1.5mm, F.Cu at (131.2, 30.7)
- added TP20: TestPoint, TestPoint:TestPoint_Pad_D1.5mm, F.Cu at (131.2, 34.2)
- added TP21: TestPoint, TestPoint:TestPoint_Pad_D1.5mm, F.Cu at (234.8, 128.1)
- added TP22: TestPoint, TestPoint:TestPoint_Pad_D1.5mm, F.Cu at (234.8, 130.6)
- added TP23: TestPoint, TestPoint:TestPoint_Pad_D1.5mm, F.Cu at (279.3, -11.5)
- added TP24: TestPoint, TestPoint:TestPoint_Pad_D1.5mm, F.Cu at (190.2, 50.6)
- added U7: TLIN2021, Package_SO:SOIC-8_5.3x5.3mm_P1.27mm, F.Cu at (293.9, -23.3)
- added Y1: ABM3BAIG, Crystal:Crystal_SMD_5032-4Pin_5.0x3.2mm, F.Cu at (202.3, 133.2)
- C28, C29: footprint Capacitor_SMD:C_1206_3216Metric -> Capacitor_SMD:C_0805_2012Metric
- D5: footprint Diode_SMD:D_SMA -> Diode_SMD:D_SMB
- L3: footprint Inductor_SMD:L_Bourns-SRN8040_8x8.15mm -> Inductor_SMD:L_APV_ANR3012
- moved Q6 242.5 mm to (320.4, 128.2)
- moved D8 238.1 mm to (314.3, 122.8)
- moved Q8 237.3 mm to (320.5, 117.0), turned to 180 degrees
- moved C42 235.1 mm to (326.8, 123.6), turned to 90 degrees
- moved Q4 234.7 mm to (314.8, 127.4), turned to 180 degrees
- moved Q12 234.2 mm to (320.8, 109.8), turned to 180 degrees
- moved R32 233.5 mm to (329.6, 122.8)
- moved R33 233.2 mm to (329.6, 124.5)
- moved D10 230.4 mm to (314.0, 106.1), turned to 180 degrees
- moved Q13 229.9 mm to (319.5, 102.1)
- moved Q7 229.0 mm to (315.1, 117.8)
- moved C43 229.0 mm to (326.6, 106.8), turned to 90 degrees
- moved R35 227.8 mm to (324.3, 128.2)
- moved R31 227.1 mm to (321.6, 122.8)
- moved R30 224.9 mm to (318.1, 122.8)
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Connections:
- C10 pad 1: Net-(U2-VIN) -> VCC
- C11 pad 1: Net-(U2-VIN) -> VCC
- C14 pad 1: Net-(C14-Pad1) -> Net-(C13-Pad2)
- C8 pad 1: Net-(U2-VIN) -> VCC
- C9 pad 1: Net-(U2-VIN) -> VCC
- L1 pad 1: Net-(U2-BST) -> Net-(U2-SW)
- L4 pad 1: /IO_Interface/CANH -> /IO_Interface/CANL
- L4 pad 2: /IO_Interface/CANL -> /IO_Interface/CANH
- L4 pad 3: Net-(U6-CANL) -> Net-(U6-CANH)
- L4 pad 4: Net-(U6-CANH) -> Net-(U6-CANL)
- Q9 pad 2: /IO_Interface/GPIO3_HI -> /mcu/GPIO3_HI
- Q9 pad 5: /IO_Interface/GPIO4_HI -> /mcu/GPIO4_HI
- R1 pad 1: Net-(U2-VIN) -> VCC
- R35 pad 2: /IO_Interface/GPIO3_LO -> /mcu/GPIO3_LO
- R43 pad 2: /IO_Interface/GPIO4_LO -> /mcu/GPIO4_LO
- R5 pad 1: Net-(U2-BST) -> Net-(U2-SW)
- R5 pad 2: Net-(C14-Pad1) -> Net-(C13-Pad2)
- R6 pad 2: Net-(C13-Pad2) -> Net-(U2-FB)
- R7 pad 1: Net-(C13-Pad2) -> Net-(U2-FB)
- U1 pad 12: unconnected-(U1B-PF0-OSC_IN-Pad12) -> Net-(U1B-PF0-OSC_IN)
- U1 pad 13: unconnected-(U1B-PF1-OSC_OUT-Pad13) -> Net-(U1B-PF1-OSC_OUT)
- U1 pad 14: unconnected-(U1B-PG10-NRST-Pad14) -> /mcu/~{RST}
- U1 pad 21: unconnected-(U1A-PA1-Pad21) -> /Power/AD_12V
- U1 pad 22: unconnected-(U1A-PA2-Pad22) -> /IO_Interface/AD_GPIO1
- U1 pad 25: unconnected-(U1A-PA3-Pad25) -> /IO_Interface/AD_GPIO2
- U1 pad 26: unconnected-(U1A-PA4-Pad26) -> /IO_Interface/AD_GPIO3
- U1 pad 27: unconnected-(U1A-PA5-Pad27) -> /mcu/AD_TEMP_INRUSH
- U1 pad 28: unconnected-(U1A-PA6-Pad28) -> /mcu/AD_TEMP_AMB
- U1 pad 29: unconnected-(U1A-PA7-Pad29) -> /mcu/AD_VCC_CURRENT
- U1 pad 34: unconnected-(U1A-PB2-Pad34) -> /mcu/LIN_PULLDOWN
- U1 pad 55: unconnected-(U1A-PD8-Pad55) -> /IO_Interface/LIN_TX
- U1 pad 56: unconnected-(U1A-PD9-Pad56) -> /IO_Interface/LIN_RX
- U1 pad 61: /mcu/CAN_STB -> /IO_Interface/CAN_STB
- U1 pad 62: unconnected-(U1A-PD15-Pad62) -> /mcu/ENA_LIN_MASTER
- U1 pad 69: unconnected-(U1A-PA8-Pad69) -> /mcu/LIN_SLEEP
- U1 pad 72: /mcu/CAN_RX -> /IO_Interface/CAN_RX
- U1 pad 73: /mcu/CAN_TX -> /IO_Interface/CAN_TX
- U1 pad 89: /mcu/ENA_INRUSH -> /Power/ENA_INRUSH
- U1 pad 9: /mcu/CAN_FAULT -> /IO_Interface/CAN_FAULT
- U1 pad 90: /mcu/SWO/JTDO -> /mcu/SWO
- U1 pad 91: /mcu/JTRST -> unconnected-(U1A-PB4-Pad91)
- U1 pad 92: /mcu/HEART_BEAT -> /IO_Interface/HEARTBEAT_mcu
- U1 pad 96: /mcu/CAN_ENA -> /IO_Interface/CAN_ENA
- U2 pad 2: Net-(U2-VIN) -> VCC
Routing:
- net Net-(U4-FB): track 0.00 -> 10.4 mm, vias 0 -> 2
- net Net-(Q7-C): track 0.00 -> 10.1 mm
- net Net-(U1B-PF0-OSC_IN): track 0.00 -> 9.44 mm
- net Net-(JP3-A): track 0.00 -> 9.09 mm
- net Net-(Q7-B): track 0.00 -> 8.39 mm
- net +3V3: track 0.00 -> 8.22 mm
- net GND: track 0.00 -> 8.21 mm
- net Net-(U1B-PF1-OSC_OUT): track 0.00 -> 7.69 mm
- net Net-(U4-EN): track 0.00 -> 6.51 mm, vias 0 -> 2
- net /IO_Interface/GPIO_4: track 0.00 -> 3.95 mm
- net Net-(U4-SW): track 0.00 -> 3.21 mm
- net Net-(FB1-Pad1): track 0.00 -> 3.20 mm
- net Net-(U6-CANL): track 0.00 -> 2.92 mm
- net Net-(U6-CANH): track 0.00 -> 2.92 mm
- net Net-(Q8-C): track 0.00 -> 1.92 mm
Other:
- board outline added: 64 x 145 mm
- copper layers 2 -> 4
- board text added: "12V"
- board text added: "3V3"
- board text added: "5V"
- board text added: "CAN"
- board text added: "GPIO Protection"
- board text added: "I/O for mcu"
- board text added: "Inrush"
- board text added: "PROG Pins!! Remember me!"

Commit message: 15-10-2026
Parts:
- removed C42, C43: 1n, Capacitor_SMD:C_0603_1608Metric
- removed C46, C47, C48: 100n, Capacitor_SMD:C_0603_1608Metric
- removed D10, D8: BAV99, Package_TO_SOT_SMD:SOT-23
- removed D11, D9: MM3Z62VB, Diode_SMD:D_SOD-323F
- removed D14, D15: SMAJ58A, Diode_SMD:D_SMA
- removed D19: BAS516, Diode_SMD:D_SOD-523
- removed E3, E4: SparkGap, Control_PCB:Sparkgap_2021-09-02
- removed Q10, Q11, Q4, Q7: BCX56, Package_TO_SOT_SMD:SOT-89-3
- removed Q12, Q13, Q6, Q8: BC846, Package_TO_SOT_SMD:SOT-23
- removed Q9: PUMH11, Package_TO_SOT_SMD:SOT-363_SC-70-6
- removed R30, R31, R40, R42: 18k, Resistor_SMD:R_0603_1608Metric
- removed R32, R44, R61: 100k, Resistor_SMD:R_0603_1608Metric
- removed R33, R45: 4k7, Resistor_SMD:R_0603_1608Metric
- removed R34, R36, R38, R39: 47, Resistor_SMD:R_0603_1608Metric
- removed R35, R43, R62: 10k, Resistor_SMD:R_0603_1608Metric
- removed R37, R41, R58: 68k, Resistor_SMD:R_0603_1608Metric
- removed R48, R49: 100, Resistor_SMD:R_1206_3216Metric
- removed R56: 47k, Resistor_SMD:R_0603_1608Metric
- removed R57: 220k, Resistor_SMD:R_0603_1608Metric
- removed TP10, TP11, TP12, TP13, TP16, TP18, TP23: TestPoint, TestPoint:TestPoint_Pad_D1.5mm
- removed U7: TLIN2021, Package_SO:SOIC-8_5.3x5.3mm_P1.27mm
- moved C12 209.4 mm to (275.2, 80.5)
- moved C13 209.4 mm to (276.1, 83.5)
- moved D1 209.4 mm to (266.6, 37.6)
- moved D2 209.4 mm to (258.4, 34.5)
- moved L1 209.4 mm to (278.6, 74.9)
- moved R2 209.4 mm to (261.1, 82.3)
- moved R4 209.4 mm to (264.6, 83.3)
- moved R6 209.4 mm to (278.2, 83.6)
- moved U2 209.4 mm to (269.3, 80.5)
- moved U4 209.4 mm to (271.0, 60.8)
- moved C10 209.4 mm to (261.5, 78.3)
- moved C11 209.4 mm to (264.0, 78.8)
- moved C14 209.4 mm to (281.6, 80.5)
- moved C15 209.4 mm to (284.0, 72.1)
- moved C16 209.4 mm to (285.7, 72.1)
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Connections:
- J2 pad 4: /IO_Interface/LIN -> unconnected-(J2-Pin_4-Pad4)
- J2 pad 5: /IO_Interface/GPIO3 -> unconnected-(J2-Pin_5-Pad5)
- J2 pad 6: /IO_Interface/GPIO4 -> unconnected-(J2-Pin_6-Pad6)
- R71 pad 2: +12V -> +5V
- U1 pad 21: /Power/AD_12V -> /Power/AD_VCC_IN
- U1 pad 26: /IO_Interface/AD_GPIO3 -> /mcu/AD_GPIO3
- U1 pad 30: unconnected-(U1A-PC4-Pad30) -> /mcu/AD_GPIO4
- U1 pad 31: unconnected-(U1A-PC5-Pad31) -> /Power/AD_VCC
- U1 pad 46: unconnected-(U1B-PE15-Pad46) -> /mcu/LED_GREEN
- U1 pad 55: /IO_Interface/LIN_TX -> /mcu/LIN_TX
- U1 pad 56: /IO_Interface/LIN_RX -> /mcu/LIN_RX
- U1 pad 58: unconnected-(U1A-PD11-Pad58) -> /mcu/LED_BLUE
- U1 pad 68: unconnected-(U1A-PC9-Pad68) -> /mcu/LED_RED
Routing:
- net Net-(Q7-C): track 10.1 -> 0.00 mm
- net Net-(Q7-B): track 8.39 -> 0.00 mm
- net /IO_Interface/GPIO_4: track 3.95 -> 0.00 mm
- net Net-(Q8-C): track 1.92 -> 0.00 mm

Commit message: Schematics mostly done
Parts:
- removed C31: 270u, Capacitor_SMD:CP_Elec_8x10.5
- removed Q1: BC846, Package_TO_SOT_SMD:SOT-23
- removed Q14: BCX56, Package_TO_SOT_SMD:SOT-89-3
- added C212: 100n, Capacitor_SMD:C_0603_1608Metric, F.Cu at (344.7, 32.3)
- added C213: 1u, Capacitor_SMD:C_0603_1608Metric, F.Cu at (344.7, 34.8)
- added C214: 100n, Capacitor_SMD:C_0603_1608Metric, F.Cu at (206.9, 82.1)
- added C215: 1u, Capacitor_SMD:C_0603_1608Metric, F.Cu at (206.9, 84.6)
- added C302: 47n, Capacitor_SMD:C_0603_1608Metric, F.Cu at (243.1, 93.1)
- added C303: 47n, Capacitor_SMD:C_0603_1608Metric, F.Cu at (243.1, 95.6)
- added C304: 47n, Capacitor_SMD:C_0603_1608Metric, F.Cu at (243.1, 98.1)
- added C305: 47u, Capacitor_SMD:CP_Elec_8x10.5, F.Cu at (299.8, 111.7)
- added D101: RED, LED_SMD:LED_0805_2012Metric, F.Cu at (338.5, 32.5)
- added D102: Green, LED_SMD:LED_0805_2012Metric, F.Cu at (338.5, 35.6)
- added D103: White, LED_SMD:LED_0805_2012Metric, F.Cu at (338.5, 38.6)
- added FB201: FerriteBead_Small, Inductor_SMD:L_0603_1608Metric, F.Cu at (306.3, 48.6)
- added Q101: MMBT3904, Package_TO_SOT_SMD:SOT-23, F.Cu at (333.8, 33.2)
- added Q102: MMBT3904, Package_TO_SOT_SMD:SOT-23, F.Cu at (333.8, 37.7)
- added Q103: MMBT3904, Package_TO_SOT_SMD:SOT-23, F.Cu at (333.8, 42.1)
- added Q301: MMBT3904, Package_TO_SOT_SMD:SOT-23, F.Cu at (333.8, 28.6)
- added Q401: MMBT3904, Package_TO_SOT_SMD:SOT-23, F.Cu at (338.5, 28.1)
- added R101: 270, Resistor_SMD:R_0603_1608Metric, F.Cu at (310.2, 28.8)
- added R102: 120, Resistor_SMD:R_0603_1608Metric, F.Cu at (310.2, 31.3)
- added R103: 120, Resistor_SMD:R_0603_1608Metric, F.Cu at (310.2, 33.8)
- added R104: 10k, Resistor_SMD:R_0603_1608Metric, F.Cu at (310.2, 36.3)
- added R105: 10k, Resistor_SMD:R_0603_1608Metric, F.Cu at (310.2, 38.8)
- added R106: 10k, Resistor_SMD:R_0603_1608Metric, F.Cu at (310.2, 41.4)
- added R207: 47, Resistor_SMD:R_0603_1608Metric, F.Cu at (316.2, 31.3)
- C204: renamed from C1; value 10u -> 22u; footprint Capacitor_SMD:C_0603_1608Metric -> Capacitor_SMD:C_0805_2012Metric
- C313: renamed from C16; value 10u -> 22u; footprint Capacitor_SMD:C_0603_1608Metric -> Capacitor_SMD:C_0805_2012Metric
- C316: renamed from C18; footprint Capacitor_SMD:C_0603_1608Metric -> Capacitor_SMD:C_0805_2012Metric
- C317: renamed from C19; footprint Capacitor_SMD:C_0603_1608Metric -> Capacitor_SMD:C_0805_2012Metric
- Q302: renamed from Q2; value NTMFS016N06CT1G -> NTMFS015N10MCLT1G
- Q303: renamed from Q3; value NTMFS016N06CT1G -> NTMFS015N10MCLT1G
- R203: renamed from R63; value 100 -> 120
- R205: renamed from R64; value 100 -> 120
- R304: renamed from R13; value 1k -> 10k
- R306: renamed from R12; value 10k -> 100k
- R316: renamed from R6; value 1k -> 390k
- R321: renamed from R7; value 1k -> 120k
- R324: renamed from R3; value 470k -> 240k
- R405: renamed from R69; value 1k -> 10k
- renumbered C49 to C201, C50 to C202, C52 to C203, C2 to C205, C3 to C206, C4 to C207, C5 to C208, C6 to C209, C7 to C210, C51 to C211, C25 to C250, C26 to C260, C28 to C280, C29 to C290, C30 to C300, C35 to C301, C34 to C306, C12 to C307, C8 to C308, C9 to C309, C10 to C310, C11 to C311, C15 to C312, C14 to C314, C24 to C315, C13 to C318, C20 to C319, C44 to C401, C45 to C402, C53 to C403, C38 to C404, C37 to C405, C36 to C406, C40 to C407, C39 to C408, C41 to C409, D21 to D201, D7 to D301, D5 to D302, D18 to D303, D17 to D304, D3 to D305, D1 to D306, D2 to D307, D12 to D401, D13 to D402, D20 to D403, D4 to D404, D16 to D405, D6 to D406, E1 to E401, E2 to E402, E5 to E403, E6 to E404, FB1 to FB100, J1 to J101, J3 to J102, J2 to J103, J4 to J201, JP3 to JP30, JP1 to JP301, JP2 to JP302, L3 to L30, L1 to L301, L2 to L302, L4 to L401, Q5 to Q304, R14 to R140, R15 to R150, R16 to R160, R68 to R201, R66 to R202, R67 to R204, R65 to R206, R11 to R301, R53 to R302, R50 to R303, R54 to R305, R51 to R307, R59 to R308, R55 to R309, R52 to R310, R60 to R311, R22 to R312, R23 to R313, R17 to R314, R1 to R315, R5 to R317, R8 to R318, R10 to R319, R2 to R320, R9 to R322, R4 to R323, R71 to R401, R46 to R402, R47 to R403, R72 to R404, R70 to R406, R20 to R407, R21 to R408, R24 to R409, R25 to R410, R18 to R411, R19 to R412, R26 to R413, R27 to R414, R28 to R415, R29 to R416, TP19 to TP201, TP21 to TP202, TP20 to TP203, TP22 to TP204, TP2 to TP301, TP14 to TP302, TP15 to TP303, TP17 to TP304, TP1 to TP305, TP3 to TP306, TP24 to TP307, TP6 to TP401, TP7 to TP402, TP4 to TP403, TP5 to TP404, TP8 to TP405, TP9 to TP406, U1 to U201, U5 to U301, U3 to U302, U2 to U303, U4 to U40, U6 to U401, Y1 to Y201
Connections:
- D303 pad 1: /Power/AD_VCC_IN -> Net-(D303-K)
- D304 pad 1: /Power/AD_VCC -> Net-(D304-K)
- R302 pad 2: Net-(R53-Pad2) -> Net-(D303-K)
- R303 pad 2: Net-(R50-Pad2) -> Net-(D304-K)
- R305 pad 1: Net-(R53-Pad2) -> Net-(D303-K)
- R307 pad 1: Net-(R50-Pad2) -> Net-(D304-K)
- U201 pad 36: unconnected-(U1C-VREF+-Pad36) -> Net-(U201C-VREF+)
