File: Control_PCB/Control_PCB.kicad_pcb (KiCad board)
At the start: 4 copper layers, 64 x 145 mm, 170 parts, among them J101 Minifit 2x3, J102 Conn_01x05, J103 Conn_01x09, J201 Micro Match, Q101 MMBT3904, Q102 MMBT3904, Q103 MMBT3904, Q301 MMBT3904, Q302 NTMFS015N10MCLT1G, Q303 NTMFS015N10MCLT1G, Q304 2N7002, Q401 MMBT3904, U201 STM32G473VET3, U301 VOM1271T, U302 TPS62A01APDDC, U303 LM5164DDA, U40 TLV61046ADB, U401 TCAN1043xDxQ1, Y201 ABM3BAIG

Commit message: Updated schematic started on layout for motor PCB
Parts:
- added C410: 47n, Capacitor_SMD:C_0603_1608Metric, F.Cu at (153.5, 60.4)
- added C411: 47n, Capacitor_SMD:C_0603_1608Metric, F.Cu at (153.5, 62.9)
- D302: footprint Diode_SMD:D_SMB -> Diode_SMD:D_SMC
- D303, D304: footprint Diode_SMD:D_SMA -> Diode_SMD:D_SOD-323F
- D305: footprint Diode_SMD:D_SOD-323 -> Diode_SMD:D_SMC
- D306: value B360 -> B360A; footprint Diode_SMD:D_SMB -> Diode_SMD:D_SMA
- J201: moved to B.Cu
- Q302, Q303: value NTMFS015N10MCLT1G -> TPH4R50ANH1; footprint Package_SO:ONSemi_SO-8FL_488AA -> Package_SON:Infineon_PG-TDSON-8_6.15x5.15mm
- R401: value 100k -> 1k
- R404: value 100k -> 100
- moved C307 77.8 mm to (201.7, 106.0)
- moved C318 77.8 mm to (202.6, 109.0)
- moved L301 77.8 mm to (205.1, 100.5)
- moved R316 77.8 mm to (204.7, 109.2)
- moved R320 77.8 mm to (187.6, 107.8)
- moved R323 77.8 mm to (191.1, 108.8)
- moved U303 77.8 mm to (195.8, 106.0)
- moved C308 77.8 mm to (179.3, 106.0)
- moved C310 77.8 mm to (188.0, 103.8)
- moved C311 77.8 mm to (190.5, 104.4)
- moved C312 77.8 mm to (210.5, 97.7)
- moved C314 77.8 mm to (208.1, 106.0)
- moved JP301 77.8 mm to (214.3, 97.8)
- moved R321 77.8 mm to (201.0, 109.5)
- moved R324 77.8 mm to (189.3, 107.8)
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
Commit message: 20/10-2026
Parts:
- removed C306: 47u, Capacitor_SMD:CP_Elec_8x10.5
- U301: footprint Package_SO:SOP-4_7.5x4.1mm_P2.54mm -> Control_PCB:SOP-4_VIS
- moved C315 113.1 mm to (120.8, 141.2)
- moved C316 113.1 mm to (112.2, 140.9)
- moved C317 113.1 mm to (113.9, 140.9)
- moved D307 113.1 mm to (107.5, 129.7)
- moved R318 113.1 mm to (116.9, 137.9)
- moved R319 113.1 mm to (107.5, 132.8)
- moved R322 113.1 mm to (120.0, 137.9)
- moved U302 113.1 mm to (117.4, 140.7)
- moved C319 113.1 mm to (104.5, 141.7)
- moved D306 113.1 mm to (115.7, 132.8)
- moved JP302 113.1 mm to (111.2, 144.1)
- moved L302 113.1 mm to (115.0, 144.1)
- moved C308 50.2 mm to (205.3, 63.0), turned to 0 degrees
- moved L401 48.2 mm to (231.1, 165.9), turned to 90 degrees
- moved R315 42.1 mm to (203.4, 69.6), turned to 180 degrees
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