File: Control_PCB/Control_PCB.kicad_sch (KiCad schematic)
At the start: 0 parts

Commit message: 02-10-2026
Other:
- added sheet IO_Interface (IO_Interface.kicad_sch)
Changed lines of the file:
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@@
 	(paper "A4")
 	(sheet
-		(at 114.3 133.35)
+		(at 96.52 113.03)
 		(size 27.94 17.78)
 		(exclude_from_sim no)
@@
 		)
 		(property "Sheetname" "Power"
-			(at 114.3 132.6384 0)
+			(at 96.52 112.3184 0)
 			(show_name no)
 			(do_not_autoplace no)
@@
 		)
 		(property "Sheetfile" "Power.kicad_sch"
-			(at 114.3 151.7146 0)
+			(at 96.52 131.3946 0)
 			(show_name no)
 			(do_not_autoplace no)
@@
 	)
 	(sheet
-		(at 160.02 39.37)
+		(at 151.13 36.83)
 		(size 26.67 60.96)
 		(exclude_from_sim no)
@@
 		)
 		(property "Sheetname" "mcu"
-			(at 160.02 38.6584 0)
+			(at 151.13 36.1184 0)
 			(show_name no)
 			(do_not_autoplace no)
@@
 		)
 		(property "Sheetfile" "mcu.kicad_sch"
-			(at 160.02 100.9146 0)
+			(at 151.13 98.3746 0)
 			(show_name no)
 			(do_not_autoplace no)
@@
 				)
 			)
+		)
+	)
+	(sheet
+		(at 81.28 43.18)
+		(size 26.67 40.64)
+		(exclude_from_sim no)
+		(in_bom yes)
+		(on_board yes)
+		(dnp no)
+		(fields_autoplaced yes)
+		(stroke
+			(width 0.1524)
+			(type solid)
+		)
+		(fill
+			(color 0 0 0 0)
+		)
+		(property "Sheetname" "IO_Interface"
+			(at 81.28 42.4684 0)
+			(show_name no)
+			(do_not_autoplace no)
+			(effects
+				(font
+					(size 1.27 1.27)
+				)
+				(justify left bottom)
+			)
+		)
+		(property "Sheetfile" "IO_Interface.kicad_sch"
+			(at 81.28 84.4046 0)
+			(show_name no)
+			(do_not_autoplace no)
+			(effects
+				(font
+					(size 1.27 1.27)
+				)
+				(justify left top)
+			)
+		)
+		(property "Field2" ""
+			(at 81.28 43.18 0)
+			(hide yes)
+			(show_name no)
+			(do_not_autoplace no)
+			(effects
+				(font
+					(size 1.27 1.27)
+				)
+			)
+		)
+		(instances
+			(project "Control_PCB"
+				(path "/dd8adfc1-6bab-46c3-a8c6-367c772462fc"
+					(page "4")
+				)
+			)

Commit message: 04-10-2026
Changed lines of the file:
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@@
 	(paper "A4")
 	(sheet
-		(at 96.52 113.03)
+		(at 80.01 92.71)
 		(size 27.94 17.78)
 		(exclude_from_sim no)
@@
 		)
 		(property "Sheetname" "Power"
-			(at 96.52 112.3184 0)
+			(at 80.01 91.9984 0)
 			(show_name no)
 			(do_not_autoplace no)
@@
 		)
 		(property "Sheetfile" "Power.kicad_sch"
-			(at 96.52 131.3946 0)
+			(at 80.01 111.0746 0)
 			(show_name no)
 			(do_not_autoplace no)

Commit message: 07-20-2026
Parts:
- added J1, J3: Minifit 2x3, Connector_Molex:Molex_Mini-Fit_Jr_5569-06A2_2x03_P4.20mm_Horizontal, symbol Connector_Generic:Conn_02x03_Counter_Clockwise
- added J2: Conn_01x09, symbol Connector_Generic:Conn_01x09
Connections:
- new net GND: J1.1 (Pin_1), J1.2 (Pin_2), J1.3 (Pin_3), J3.1 (Pin_1), J3.2 (Pin_2)
- new net IO_Interface/LIN: J2.4 (Pin_4)
- new net VCC_IN: J1.4 (Pin_4), J1.5 (Pin_5), J1.6 (Pin_6), J3.5 (Pin_5), J3.6 (Pin_6)
Other:
- sheet IO_Interface ports: added AD_GPIO1, AD_GPIO2, AD_GPIO3, AD_GPIO4, CANH, CANL, CAN_ENA, CAN_FAULT, CAN_RX, CAN_STB, CAN_TX, GPIO1, GPIO2, GPIO3, GPIO3_HI, GPIO3_LO, GPIO4, GPIO4_HI, GPIO4_LO, LIN, LIN_RX, LIN_TX; removed none
- sheet Power ports: added AD_12V, AD_5V, AD_VCC, AD_VCC_IN, ENA_INRUSH; removed none
- sheet mcu ports: added AD_12V, AD_5V, AD_GPIO1, AD_GPIO2, AD_GPIO3, CAN_ENA, CAN_FAULT, CAN_RX, CAN_STB, CAN_TX, ENA_INRUSH, GPIO3_HI, GPIO3_LO, GPIO4_HI, GPIO4_LO, LIN_RX, LIN_TX; removed none
- note added: "Black"
- note added: "GPIO1"
- note added: "GPIO2"
- note added: "GPIO3"
- note added: "GPIO4"
- note added: "Green"
- note added: "Grey"
- note added: "LIN"
- note added: "LIN GND"
- note added: "Light_blue"
- note added: "Orange"
- note added: "Purple"
- note added: "Red"
- note added: "White"
- note added: "Yellow"

Commit message: 10-10-2026
Parts:
- removed J3: Minifit 2x3, Connector_Molex:Molex_Mini-Fit_Jr_5569-06A2_2x03_P4.20mm_Horizontal, symbol Connector_Generic:Conn_02x03_Counter_Clockwise
- added J5: Conn_01x04_Shielded, Package_DIP:DIP-20_W7.62mm, symbol Connector_Generic_Shielded:Conn_01x04_Shielded
Connections:
- net CANH: now also J5.2 (Pin_2)
- net CANL: now also J5.3 (Pin_3)
- net GND: now also J5.4 (Pin_4)

Commit message: Before removing stuffs
Parts:
- removed J5: Conn_01x04_Shielded, Package_DIP:DIP-20_W7.62mm, symbol Connector_Generic_Shielded:Conn_01x04_Shielded
- added J3: Conn_01x05, Control_PCB:1411976, symbol Connector_Generic:Conn_01x05
- J2: footprint (none) -> Control_PCB:Molex_Micro-Fit_3x03_P3.00mm
Connections:
- net GND: now also J2.3 (Pin_3), J3.1 (Pin_1), J3.3 (Pin_3)
- net IO_Interface/CANH: now also J3.4 (Pin_4)
- net IO_Interface/CANL: now also J3.5 (Pin_5)
- net IO_Interface/GPIO1: now also J2.7 (Pin_7)
- net IO_Interface/GPIO2: now also J2.8 (Pin_8)
- net IO_Interface/GPIO3: now also J2.5 (Pin_5)
- net IO_Interface/GPIO4: now also J2.6 (Pin_6)
- new net IO_Interface/HEARTBEAT: J3.2 (Pin_2)
Other:
- sheet IO_Interface ports: added HEARTBEAT, HEARTBEAT_mcu; removed none
- sheet mcu ports: added HEARTBEAT_mcu; removed none
- note added: "CANH"
- note added: "CANL"
- note added: "Heartbeat"
- note added: "Optional Shield"
- note added: "Pinout based on CANOPEN CiA DR-303-1 Page: 14 https://affon.narod.ru/CAN/DR303_1.pdf"
- moved on the sheet: J1, J2

Commit message: 15-10-2026
Connections:
- net IO_Interface/GPIO3: no longer names the net of J2.5 (Pin_5)
- net IO_Interface/GPIO4: no longer names the net of J2.6 (Pin_6)
- net IO_Interface/LIN: no longer names the net of J2.4 (Pin_4)
- no-connect marks 0 -> 15
Other:
- sheet IO_Interface ports: added none; removed AD_GPIO3, AD_GPIO4, GPIO3, GPIO3_HI, GPIO3_LO, GPIO4, GPIO4_HI, GPIO4_LO, LIN, LIN_RX, LIN_TX
- sheet Power ports: added none; removed AD_12V
- sheet mcu ports: added AD_GPIO4, AD_VCC, ENA_LIN_MASTER; removed none
- moved on the sheet: J1, J2, J3

Commit message: Schematics mostly done
Parts:
- added D101: RED, LED_SMD:LED_0805_2012Metric, symbol Device:LED
- added D102: Green, LED_SMD:LED_0805_2012Metric, symbol Device:LED
- added D103: White, LED_SMD:LED_0805_2012Metric, symbol Device:LED
- added Q101, Q102, Q103: MMBT3904, Package_TO_SOT_SMD:SOT-23, symbol Transistor_BJT:MMBT3904
- added R101: 270, Resistor_SMD:R_0603_1608Metric, symbol Device:R_Small
- added R102, R103: 120, Resistor_SMD:R_0603_1608Metric, symbol Device:R_Small
- added R104, R105, R106: 10k, Resistor_SMD:R_0603_1608Metric, symbol Device:R_Small
- renumbered J1 to J101, J3 to J102, J2 to J103
Connections:
- net GND: now also Q101.2 (E), Q102.2 (E), Q103.2 (E)
- new net: Q101.3 (C), R101.1
- new net: D101.1 (K), R101.2
- new net: Q103.1 (B), R106.1
- new net: Q103.3 (C), R103.1
- new net: Q101.1 (B), R104.1
- new net: D103.1 (K), R103.2
- new net: Q102.3 (C), R102.1
- new net: D102.1 (K), R102.2
- new net: Q102.1 (B), R105.1
- new net +5V: D101.2 (A), D102.2 (A), D103.2 (A)
- new net mcu/LED_BLUE: R106.2
- new net mcu/LED_GREEN: R105.2
- new net mcu/LED_RED: R104.2
Other:
- sheet mcu ports: added LED_BLUE, LED_GREEN, LED_RED; removed none
- note added: "TO DO: UPDATE MOSFETS AND FOOTPRINT TO THE ONE ON THE MOTOR PCB!!! ADD BACK THE LIN TRANCEIVER"
- moved on the sheet: J101

Commit message: 20/10-2026
Other:
- note removed: "TO DO: UPDATE MOSFETS AND FOOTPRINT TO THE ONE ON THE MOTOR PCB!!! ADD BACK THE LIN TRANCEIVER"
Changed lines of the file:
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@@
-		)
-	)
-	(text "TO DO: \nUPDATE MOSFETS AND FOOTPRINT TO THE ONE ON THE MOTOR PCB!!!\nADD BACK THE LIN TRANCEIVER"
-		(exclude_from_sim no)
-		(at 111.76 20.32 0)
-		(effects
-			(font
-				(size 2.032 2.032)
-				(thickness 0.4064)
-				(bold yes)
-			)
-			(justify left)
 		)
 	)
