File: Motor_PCB/Motor_PCB.kicad_sch (KiCad schematic)
At the start: 12 parts, among them U6 TCAN1043xDxQ1

Commit message: 10-10-2026
Parts:
- added C1: 100n, Diode_SMD:D_SMB, symbol Device:C_Small
- added C2: 150n, Diode_SMD:D_SMB, symbol Device:C_Small
- added C3: 2.2u, Diode_SMD:D_SMB, symbol Device:C_Small
- added D2: SM6T15A, Diode_SMD:D_SMB, symbol Diode:SM6T15A
- added D3, D4: D, Package_TO_SOT_SMD:SOT-23, symbol Device:D
- added Q1: 2N7002, Package_TO_SOT_SMD:SOT-23, symbol Transistor_FET:2N7002
- added Q2: BC856, Package_TO_SOT_SMD:SOT-23, symbol Transistor_BJT:BC856
- added R2: 100k, Resistor_THT:R_Array_SIP4, symbol Device:R_Small
- added R3: 39k, Resistor_THT:R_Array_SIP4, symbol Device:R_Small
- added R4, R6, R7: 10k, Resistor_THT:R_Array_SIP4, symbol Device:R_Small
- added R5: 470k, Resistor_THT:R_Array_SIP4, symbol Device:R_Small
Connections:
- net +3V3: now also C3.1, D3.1 (K), Q2.3 (C), R4.2, R5.2
- net GND: now also C1.2, D2.2 (A2), Q1.2 (S), R3.1, R7.1
- new net: Q2.1 (B), R6.2
- new net: C2.2, D3.2 (A), D4.1 (K)
- new net: C2.1, Q1.3 (D), R4.1
- new net: C3.2, D4.2 (A), R5.1, R6.1
- new net: Q1.1 (G), R2.2, R3.2
- new net Heatbeat_input: C1.1, D2.1 (A1), R2.1
- new net SAFE_ENA_HBRIDGE: Q2.2 (E), R7.2
Other:
- added sheet STSpin (STSpin.kicad_sch)
- note added: "HEATBEAT"
- moved on the sheet: C36, C37, C38, C39, D1, R1, R18, R19, R20, TP4, TP5, U6

Commit message: 15-10-2026
Parts:
- added C31: 270u, Capacitor_SMD:CP_Elec_8x10.5, symbol Device:C_Polarized_Small
- added C34: 47u, Capacitor_SMD:CP_Elec_8x10.5, symbol Device:C_Polarized_Small
- added C35: 10n, Capacitor_SMD:C_0603_1608Metric, symbol Device:C_Small
- added D5: S3M-13-F, Diode_SMD:D_SOD-323, symbol Device:D
- added D7: MM5Z12V, Diode_SMD:D_SOD-523, symbol Diode:MM5Zxx
- added Q3: BC846, Package_TO_SOT_SMD:SOT-23, symbol Transistor_BJT:BC846
- added Q4, Q6: NTMFS016N06CT1G, Package_SO:ONSemi_SO-8FL_488AA, symbol Transistor_FET:NTMFS016N06CT1G
- added Q5: 2N7002, Package_TO_SOT_SMD:SOT-23, symbol Transistor_FET:2N7002
- added R11: 200, Resistor_SMD:R_0603_1608Metric, symbol Device:R_Small
- added R12: 10k, Resistor_SMD:R_0603_1608Metric, symbol Device:R_Small
- added R13: 1k, Resistor_SMD:R_0603_1608Metric, symbol Device:R_Small
- added R17: 47R - 3W, Resistor_SMD:R_2512_6332Metric, symbol Device:R
- added R22: 1Meg, Resistor_SMD:R_0603_1608Metric, symbol Device:R_Small
- added R23: 100k, Resistor_SMD:R_0603_1608Metric, symbol Device:R_Small
- added TP1, TP2, TP24, TP3: TestPoint, TestPoint:TestPoint_Pad_D1.5mm, symbol Connector:TestPoint
- added U5: VOM1271T, Package_SO:SOP-4_7.5x4.1mm_P2.54mm, symbol Control_PCB:Photovoltaic
Connections:
- net +3V3: now also U5.1
- net GND: now also C31.2, C34.2, Q5.2 (S), R12.2, R23.1
- net VCC: now also C31.1, C34.1, Q6.5 (D), R17.2, TP1.1
- new net: C35.2, D7.2 (A), Q4.1 (S), Q4.2 (S), Q4.3 (S), Q6.1 (S), Q6.2 (S), Q6.3 (S), TP3.1, U5.3
- new net: C35.1, D7.1 (K), Q4.4 (G), Q6.4 (G), TP2.1, U5.4
- new net: D5.1 (K), R17.1
- new net: Q3.1 (B), R12.1, R13.2
- new net: Q5.1 (G), R22.2, R23.2
- new net: Q3.2 (E), Q5.3 (D)
- new net: R11.1, U5.2
- new net: Q3.3 (C), R11.2
- new net ENA_INRUSH: R13.1
- new net VCC_IN: D5.2 (A), Q4.5 (D), R22.1, TP24.1
Other:
- added sheet Inverter (Inverter.kicad_sch)
- note added: "+8V"
- note added: "Change the FETS to something rated for higher voltages!!! Also look at R_ON at 7V V_GS"
- note added: "Inrush Protection Reverse Protection"
- note added: "≈ 17 mΩ @ 7V V_GS"

Commit message: Schematics mostly done
Parts:
- removed C1: 100n, Diode_SMD:D_SMB, symbol Device:C_Small
- removed C2: 150n, Diode_SMD:D_SMB, symbol Device:C_Small
- removed C3: 2.2u, Diode_SMD:D_SMB, symbol Device:C_Small
- removed C31: 270u, Capacitor_SMD:CP_Elec_8x10.5, symbol Device:C_Polarized_Small
- removed C34: 47u, Capacitor_SMD:CP_Elec_8x10.5, symbol Device:C_Polarized_Small
- removed C35: 10n, Capacitor_SMD:C_0603_1608Metric, symbol Device:C_Small
- removed C36, C37, C38: 100n, Capacitor_SMD:C_0603_1608Metric, symbol Device:C_Small
- removed C39: 4.7n, Capacitor_SMD:C_0603_1608Metric, symbol Device:C_Small
- removed D1: MM1Z62, Diode_SMD:Littelfuse_PolyZen-LS, symbol Device:D_Zener
- removed D2: SM6T15A, Diode_SMD:D_SMB, symbol Diode:SM6T15A
- removed D3, D4: D, Package_TO_SOT_SMD:SOT-23, symbol Device:D
- removed D5: S3M-13-F, Diode_SMD:D_SOD-323, symbol Device:D
- removed D7: MM5Z12V, Diode_SMD:D_SOD-523, symbol Diode:MM5Zxx
- removed Q1, Q5: 2N7002, Package_TO_SOT_SMD:SOT-23, symbol Transistor_FET:2N7002
- removed Q2: BC856, Package_TO_SOT_SMD:SOT-23, symbol Transistor_BJT:BC856
- removed Q3: BC846, Package_TO_SOT_SMD:SOT-23, symbol Transistor_BJT:BC846
- removed Q4, Q6: NTMFS016N06CT1G, Package_SO:ONSemi_SO-8FL_488AA, symbol Transistor_FET:NTMFS016N06CT1G
- removed R1: 4K7, Resistor_THT:R_Array_SIP4, symbol Device:R_Small
- removed R11: 200, Resistor_SMD:R_0603_1608Metric, symbol Device:R_Small
- removed R12: 10k, Resistor_SMD:R_0603_1608Metric, symbol Device:R_Small
- removed R13: 1k, Resistor_SMD:R_0603_1608Metric, symbol Device:R_Small
- removed R17: 47R - 3W, Resistor_SMD:R_2512_6332Metric, symbol Device:R
- removed R18, R19, R20: 60, Resistor_SMD:R_0603_1608Metric, symbol Device:R_Small
- removed R2: 100k, Resistor_THT:R_Array_SIP4, symbol Device:R_Small
- removed R22: 1Meg, Resistor_SMD:R_0603_1608Metric, symbol Device:R_Small
- removed R23: 100k, Resistor_SMD:R_0603_1608Metric, symbol Device:R_Small
- removed R3: 39k, Resistor_THT:R_Array_SIP4, symbol Device:R_Small
- removed R4, R6, R7: 10k, Resistor_THT:R_Array_SIP4, symbol Device:R_Small
- removed R5: 470k, Resistor_THT:R_Array_SIP4, symbol Device:R_Small
- removed TP1, TP2, TP24, TP3, TP4, TP5: TestPoint, TestPoint:TestPoint_Pad_D1.5mm, symbol Connector:TestPoint
- removed U5: VOM1271T, Package_SO:SOP-4_7.5x4.1mm_P2.54mm, symbol Control_PCB:Photovoltaic
- removed U6: TCAN1043xDxQ1, Package_SO:SOIC-14_3.9x8.7mm_P1.27mm, symbol Interface_CAN_LIN:TCAN1043xDxQ1
- added D101: RED, LED_SMD:LED_0805_2012Metric, symbol Device:LED
- added D102: Green, LED_SMD:LED_0805_2012Metric, symbol Device:LED
- added D103: White, LED_SMD:LED_0805_2012Metric, symbol Device:LED
- added J101: Conn_01x05, MOTOR_PCB:1411976, symbol Connector_Generic:Conn_01x05
- added J102: Conn_01x03_Pin, Connector_Wire:SolderWire-1.5sqmm_1x03_P6mm_D1.7mm_OD3mm, symbol Connector:Conn_01x03_Pin
- added J103: Conn_01x03_Pin, symbol Connector:Conn_01x03_Pin
- added J104: Minifit 2x3, Connector_Molex:Molex_Mini-Fit_Jr_5569-06A2_2x03_P4.20mm_Horizontal, symbol Connector_Generic:Conn_02x03_Counter_Clockwise
- added J105, J106: Conn_01x06, symbol Connector_Generic:Conn_01x06
- added Q101, Q102, Q103: MMBT3904, Package_TO_SOT_SMD:SOT-23, symbol Transistor_BJT:MMBT3904
- added R101: 270, Resistor_SMD:R_0603_1608Metric, symbol Device:R_Small
- added R102, R103: 120, Resistor_SMD:R_0603_1608Metric, symbol Device:R_Small
- added R104, R105, R106: 10k, Resistor_SMD:R_0603_1608Metric, symbol Device:R_Small
Connections:
- net +5V: now also D101.2 (A), D102.2 (A), D103.2 (A), J105.4 (Pin_4), J106.4 (Pin_4)
- net GND: now also J101.1 (Pin_1), J101.3 (Pin_3), J104.1 (Pin_1), J104.2 (Pin_2), J104.3 (Pin_3), J105.5 (Pin_5), J106.5 (Pin_5), Q101.2 (E), Q102.2 (E), Q103.2 (E)
- new net: D102.1 (K), R102.2
- new net: Q103.1 (B), R106.1
- new net: Q103.3 (C), R103.1
- new net: D103.1 (K), R103.2
- new net: Q102.3 (C), R102.1
- new net: Q101.1 (B), R104.1
- new net: Q101.3 (C), R101.1
- new net: Q102.1 (B), R105.1
- new net: D101.1 (K), R101.2
- new net AD_TEMP: J105.6 (Pin_6), J106.6 (Pin_6)
- new net HALL_U: J105.1 (Pin_1), J106.1 (Pin_1)
- new net HALL_V: J105.2 (Pin_2), J106.2 (Pin_2)
- new net HALL_W: J105.3 (Pin_3), J106.3 (Pin_3)
- new net IO/CANH: J101.4 (Pin_4)
- new net IO/CANL: J101.5 (Pin_5)
- new net IO/HEARTBEAT_IN: J101.2 (Pin_2)
- new net LED_GREEN: R105.2
- new net LED_RED: R104.2
- new net LED_WHITE: R106.2
- new net MOTOR_U: J102.3 (Pin_3), J103.3 (Pin_3)
- new net MOTOR_V: J102.2 (Pin_2), J103.2 (Pin_2)
- new net MOTOR_W: J102.1 (Pin_1), J103.1 (Pin_1)
- new net VBUS_IN: J104.4 (Pin_4), J104.5 (Pin_5), J104.6 (Pin_6)
Other:
- added sheet IO (IO.kicad_sch)
- sheet Inverter ports: added GHS1, GHS2, GHS3, GLS1, GLS2, GLS3, PHASE_U, PHASE_V, PHASE_W, U, V, V_SHUNT_U_N, V_SHUNT_U_P, V_SHUNT_V_N, V_SHUNT_V_P, V_SHUNT_W_N, V_SHUNT_W_P, W; removed none
- sheet STSpin ports: added AD_TEMP, CAN_ENA, CAN_FAULT, CAN_RX, CAN_STB, CAN_TX, ENA_INRUSH, GHS1, GHS2, GHS3, GLS1, GLS2, GLS3, HALL_U, HALL_V, HALL_W, HEARTBEAT, LED_BLUE, LED_GREEN, LED_RED, MOTOR_U, MOTOR_V, MOTOR_W, PHASE_U, PHASE_V, PHASE_W, V_SHUNT_U_N, V_SHUNT_U_P, V_SHUNT_V_N, V_SHUNT_V_P, V_SHUNT_W_N, V_SHUNT_W_P, WAKE; removed none
- note added: "CANH"
- note added: "CANL"
- note added: "Direct Solder"
- note added: "Heartbeat"
- note added: "LEDS"
- note added: "Micro Match"
- note added: "Motor Sensors"
- note added: "Optional Shield"
- note added: "Pinout based on CANOPEN CiA DR-303-1 Page: 14 https://affon.narod.ru/CAN/DR303_1.pdf"
- note added: "Quick-disconnects"
- note removed: "+8V"
- note removed: "CAN"
- note removed: "Change the FETS to something rated for higher voltages!!! Also look at R_ON at 7V V_GS"
- note removed: "HEATBEAT"
- note removed: "Inrush Protection Reverse Protection"
- note removed: "≈ 17 mΩ @ 7V V_GS"

Commit message: Fixed some Schematic mistakes
- Fixed mirroers FETS
- Added voltage divider to TCAN INH
- fixed other minor mistakes
Parts:
- added D104: SMDJ58CA, Diode_SMD:D_SMC, symbol Diode:SMAJ58CA
- R101: value 270 -> 560
- R102, R103: value 120 -> 390
Connections:
- net GND: now also D104.1 (A1)
- net VBUS_IN: now also D104.2 (A2)
Other:
- note added: "Input Clamping"
- note added: "Power IN"
- moved on the sheet: J104

Commit message: Surely i didnt miss anything else on the schematc...
Parts:
- J104: footprint Connector_Molex:Molex_Mini-Fit_Jr_5569-06A2_2x03_P4.20mm_Horizontal -> Connector_Molex:Molex_Mini-Fit_Jr_5566-06A_2x03_P4.20mm_Vertical
- J106: footprint (none) -> MOTOR_PCB:CONN6_7-188275-6_TEC
Changed lines of the file:
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@@
 			)
 		)
-		(property "Footprint" "Connector_Molex:Molex_Mini-Fit_Jr_5569-06A2_2x03_P4.20mm_Horizontal"
+		(property "Footprint" "Connector_Molex:Molex_Mini-Fit_Jr_5566-06A_2x03_P4.20mm_Vertical"
 			(at 25.4 121.285 0)
 			(hide yes)
@@
 			)
 		)
-		(property "Footprint" ""
+		(property "Footprint" "MOTOR_PCB:CONN6_7-188275-6_TEC"
 			(at 231.14 109.22 0)
 			(hide yes)

Commit message: Updated schematic started on layout for motor PCB
Parts:
- removed J103: Conn_01x03_Pin, symbol Connector:Conn_01x03_Pin
- J105: footprint (none) -> Connector_PinHeader_1.27mm:PinHeader_1x06_P1.27mm_Vertical
Other:
- note removed: "Quick-disconnects"
- moved on the sheet: D104, J104

Commit message: 20/10-2026
Parts:
- added J103: Conn_01x05, MOTOR_PCB:1411976, symbol Connector_Generic:Conn_01x05
Connections:
- net GND: now also J103.1 (Pin_1), J103.3 (Pin_3)
- net IO/CANH renamed CANH
- net CANH: now also J103.4 (Pin_4)
- net IO/CANL renamed CANL
- net CANL: now also J103.5 (Pin_5)
- net IO/HEARTBEAT_IN renamed heatbeat
- net heatbeat: now also J103.2 (Pin_2)
Other:
- note removed: "Pinout based on CANOPEN CiA DR-303-1 Page: 14 https://affon.narod.ru/CAN/DR303_1.pdf"
- moved on the sheet: D101, D102, D103, D104, J104, J105, J106, Q101, Q102, Q103, R101, R102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
