File: Motor_PCB/Inverter.kicad_sch (KiCad schematic)
At the start: 0 parts

Commit message: Schematics mostly done
Parts:
- added C301, C302, C303: 1u, Capacitor_SMD:CP_Elec_8x10.5, symbol Device:C_Polarized_Small
- added JP301, JP302: SolderJumper_2_Open, Jumper:SolderJumper-2_P1.3mm_Open_Pad1.0x1.5mm, symbol Jumper:SolderJumper_2_Open
- added NT301, NT302, NT303: NetTie_2, NetTie:NetTie-2_SMD_Pad0.5mm, symbol Device:NetTie_2
- added Q301, Q302, Q303, Q304, Q305, Q306: TPH4R50ANH1, Package_SON:Infineon_PG-TDSON-8_6.15x5.15mm, symbol Transistor_FET:NTMFS016N06CT1G
- added R301, R302, R303, R304, R305, R306: 33, symbol Device:R_Small
- added R307, R308, R309: R_Shunt, symbol Device:R_Shunt
- added TP301, TP302, TP303, TP304, TP305, TP306, TP307, TP308, TP309, TP310, TP311, TP312: TestPoint, TestPoint:TestPoint_Pad_D1.5mm, symbol Connector:TestPoint
Connections:
- new net: C302.2, JP301.2 (B), JP302.1 (A), Q305.5 (D), R308.1, TP311.1
- new net: Q301.4 (G), R301.2, TP301.1
- new net: Q305.4 (G), R305.2, TP308.1
- new net: Q303.4 (G), R303.2, TP303.1
- new net: C301.2, JP301.1 (A), Q304.5 (D), R307.1, TP310.1
- new net: Q306.4 (G), R306.2, TP309.1
- new net: C303.2, JP302.2 (B), Q306.5 (D), R309.1, TP312.1
- new net: Q304.4 (G), R304.2, TP307.1
- new net: Q302.4 (G), R302.2, TP302.1
- new net GHS1: R301.1
- new net GHS2: R302.1
- new net GHS3: R303.1
- new net GLS1: R304.1
- new net GLS2: R305.1
- new net GLS3: R306.1
- new net GND: R307.4, R308.4, R309.4
- new net PHASE_U: NT301.1
- new net PHASE_V: NT302.1
- new net PHASE_W: NT303.1
- new net U: NT301.2, Q301.5 (D), Q304.1 (S), Q304.2 (S), Q304.3 (S), TP304.1
- new net V: NT302.2, Q302.5 (D), Q305.1 (S), Q305.2 (S), Q305.3 (S), TP305.1
- new net VBUS: C301.1, C302.1, C303.1, Q301.1 (S), Q301.2 (S), Q301.3 (S), Q302.1 (S), Q302.2 (S), Q302.3 (S), Q303.1 (S), Q303.2 (S), Q303.3 (S)
- new net V_SHUNT_U_N: R307.3
- new net V_SHUNT_U_P: R307.2
- new net V_SHUNT_V_N: R308.3
- new net V_SHUNT_V_P: R308.2
- new net V_SHUNT_W_N: R309.3
- new net V_SHUNT_W_P: R309.2
- new net W: NT303.2, Q303.5 (D), Q306.1 (S), Q306.2 (S), Q306.3 (S), TP306.1

Commit message: Fixed some Schematic mistakes
- Fixed mirroers FETS
- Added voltage divider to TCAN INH
- fixed other minor mistakes
Parts:
- C301, C302, C303: footprint Capacitor_SMD:CP_Elec_8x10.5 -> Capacitor_SMD:C_0805_2012Metric; symbol Device:C_Polarized_Small -> Device:C_Small
- R301, R302, R303, R304, R305, R306: footprint (none) -> Resistor_SMD:R_0603_1608Metric
- R307, R308: value R_Shunt -> 5m; footprint (none) -> MOTOR_PCB:R_2512_Shunt
- R309: value R_Shunt -> 4m; footprint (none) -> MOTOR_PCB:R_2512_Shunt
Connections:
- net U: now also Q301.1 (S), Q301.2 (S), Q301.3 (S), Q304.5 (D); no longer Q301.5 (D), Q304.1 (S), Q304.2 (S), Q304.3 (S)
- net V: now also Q302.1 (S), Q302.2 (S), Q302.3 (S), Q305.5 (D); no longer Q302.5 (D), Q305.1 (S), Q305.2 (S), Q305.3 (S)
- net VBUS: now also Q301.5 (D), Q302.5 (D), Q303.5 (D); no longer Q301.1 (S), Q301.2 (S), Q301.3 (S), Q302.1 (S), Q302.2 (S), Q302.3 (S), Q303.1 (S), Q303.2 (S), Q303.3 (S)
- net W: now also Q303.1 (S), Q303.2 (S), Q303.3 (S), Q306.5 (D); no longer Q303.5 (D), Q306.1 (S), Q306.2 (S), Q306.3 (S)
- net at C302.2, JP301.2 (B), JP302.1 (A)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: now also Q305.1 (S), Q305.2 (S), Q305.3 (S); no longer Q305.5 (D)
- net at C301.2, JP301.1 (A), R307.1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: now also Q304.1 (S), Q304.2 (S), Q304.3 (S); no longer Q304.5 (D)
- net at C303.2, JP302.2 (B), R309.1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: now also Q306.1 (S), Q306.2 (S), Q306.3 (S); no longer Q306.5 (D)
Changed lines of the file:
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@@
 	)
 	(symbol
-		(lib_id "Device:C_Polarized_Small")
+		(lib_id "Device:C_Small")
 		(at 160.02 87.63 0)
 		(unit 1)
@@
 			)
 		)
-		(property "Footprint" "Capacitor_SMD:CP_Elec_8x10.5"
+		(property "Footprint" "Capacitor_SMD:C_0805_2012Metric"
 			(at 160.02 87.63 0)
 			(hide yes)
@@
 			)
 		)
-		(property "Description" "Polarized capacitor, small symbol"
+		(property "Description" "Unpolarized capacitor, small symbol"
 			(at 160.02 87.63 0)
 			(hide yes)
@@
 		(lib_id "Transistor_FET:NTMFS016N06CT1G")
 		(at 74.93 71.12 0)
-		(mirror x)
 		(unit 1)
 		(body_style 1)
@@
 		)
 		(property "Footprint" "Package_SON:Infineon_PG-TDSON-8_6.15x5.15mm"
-			(at 80.01 69.215 0)
+			(at 80.01 73.025 0)
 			(hide yes)
 			(show_name no)
@@
 		)
 		(property "Datasheet" "https://www.onsemi.cn/download/data-sheet/pdf/ntmfs015n10mcl-d.pdf"
-			(at 80.01 67.31 0)
+			(at 80.01 74.93 0)
 			(hide yes)
 			(show_name no)
@@
 		(lib_id "Transistor_FET:NTMFS016N06CT1G")
 		(at 207.01 71.12 0)
-		(mirror x)
 		(unit 1)
 		(body_style 1)
@@
 		)
 		(property "Footprint" "Package_SON:Infineon_PG-TDSON-8_6.15x5.15mm"
-			(at 212.09 69.215 0)
+			(at 212.09 73.025 0)
 			(hide yes)
 			(show_name no)
@@
 		)
 		(property "Datasheet" "https://www.onsemi.cn/download/data-sheet/pdf/ntmfs015n10mcl-d.pdf"
-			(at 212.09 67.31 0)
+			(at 212.09 74.93 0)
 			(hide yes)
 			(show_name no)
@@
 			)
 		)
-		(property "Footprint" ""
+		(property "Footprint" "Resistor_SMD:R_0603_1608Metric"
 			(at 194.31 102.87 0)
 			(hide yes)
@@
 	)
 	(symbol
-		(lib_id "Device:C_Polarized_Small")
+		(lib_id "Device:C_Small")
 		(at 226.06 87.63 0)
 		(unit 1)
@@
 			)
 		)
-		(property "Footprint" "Capacitor_SMD:CP_Elec_8x10.5"
+		(property "Footprint" "Capacitor_SMD:C_0805_2012Metric"
 			(at 226.06 87.63 0)
 			(hide yes)
@@
 			)
 		)
-		(property "Description" "Polarized capacitor, small symbol"
+		(property "Description" "Unpolarized capacitor, small symbol"
 			(at 226.06 87.63 0)
 			(hide yes)
@@
 			)
 		)
-		(property "Footprint" ""
+		(property "Footprint" "Resistor_SMD:R_0603_1608Metric"
 			(at 128.27 102.87 0)
 			(hide yes)
@@
 		(lib_id "Transistor_FET:NTMFS016N06CT1G")
 		(at 207.01 102.87 0)
-		(mirror x)
 		(unit 1)
 		(body_style 1)
@@
 		)
 		(property "Footprint" "Package_SON:Infineon_PG-TDSON-8_6.15x5.15mm"
-			(at 212.09 100.965 0)
+			(at 212.09 104.775 0)
 			(hide yes)
 			(show_name no)
@@
 		)
 		(property "Datasheet" "https://www.onsemi.cn/download/data-sheet/pdf/ntmfs015n10mcl-d.pdf"
-			(at 212.09 99.06 0)
+			(at 212.09 106.68 0)
 			(hide yes)
 			(show_name no)
@@
 			)
 		)
-		(property "Value" "R_Shunt"
+		(property "Value" "4m"
 			(at 212.09 128.2699 0)
 			(show_name no)
@@
 			)
 		)
-		(property "Footprint" ""
+		(property "Footprint" "MOTOR_PCB:R_2512_Shunt"
 			(at 211.328 127 90)
 			(hide yes)
@@
 			)
 		)
-		(property "Value" "R_Shunt"
+		(property "Value" "5m"
 			(at 80.01 128.2699 0)
 			(show_name no)
@@
 			)
 		)
-		(property "Footprint" ""
+		(property "Footprint" "MOTOR_PCB:R_2512_Shunt"
 			(at 79.248 127 90)
 			(hide yes)
@@
 			)
 		)
-		(property "Footprint" ""
+		(property "Footprint" "Resistor_SMD:R_0603_1608Metric"
 			(at 62.23 102.87 0)
 			(hide yes)
@@
 			)
 		)
-		(property "Value" "R_Shunt"
+		(property "Value" "5m"
 			(at 146.05 128.2699 0)
 			(show_name no)
@@
 			)
 		)
-		(property "Footprint" ""
+		(property "Footprint" "MOTOR_PCB:R_2512_Shunt"
 			(at 145.288 127 90)
 			(hide yes)
@@
 		(lib_id "Transistor_FET:NTMFS016N06CT1G")
 		(at 74.93 102.87 0)
-		(mirror x)
 		(unit 1)
 		(body_style 1)
@@
 		)
 		(property "Footprint" "Package_SON:Infineon_PG-TDSON-8_6.15x5.15mm"
-			(at 80.01 100.965 0)
+			(at 80.01 104.775 0)
 			(hide yes)
 			(show_name no)
@@
 		)
 		(property "Datasheet" "https://www.onsemi.cn/download/data-sheet/pdf/ntmfs015n10mcl-d.pdf"
-			(at 80.01 99.06 0)
+			(at 80.01 106.68 0)
 			(hide yes)
 			(show_name no)
@@
 			)
 		)
-		(property "Footprint" ""
+		(property "Footprint" "Resistor_SMD:R_0603_1608Metric"
 			(at 194.31 71.12 0)
 			(hide yes)
@@
 			)
 		)
-		(property "Footprint" ""
+		(property "Footprint" "Resistor_SMD:R_0603_1608Metric"
 			(at 128.27 71.12 0)
 			(hide yes)
@@
 		(lib_id "Transistor_FET:NTMFS016N06CT1G")
 		(at 140.97 71.12 0)
-		(mirror x)
 		(unit 1)
 		(body_style 1)
@@
 		)
 		(property "Footprint" "Package_SON:Infineon_PG-TDSON-8_6.15x5.15mm"
-			(at 146.05 69.215 0)
+			(at 146.05 73.025 0)
 			(hide yes)
 			(show_name no)
@@
 		)
 		(property "Datasheet" "https://www.onsemi.cn/download/data-sheet/pdf/ntmfs015n10mcl-d.pdf"
-			(at 146.05 67.31 0)
+			(at 146.05 74.93 0)
 			(hide yes)
 			(show_name no)
@@
 			)
 		)
-		(property "Footprint" ""
+		(property "Footprint" "Resistor_SMD:R_0603_1608Metric"
 			(at 62.23 71.12 0)
 			(hide yes)
@@
 	)
 	(symbol
-		(lib_id "Device:C_Polarized_Small")
+		(lib_id "Device:C_Small")
 		(at 93.98 87.63 0)
 		(unit 1)
@@
 			)
 		)
-		(property "Footprint" "Capacitor_SMD:CP_Elec_8x10.5"
+		(property "Footprint" "Capacitor_SMD:C_0805_2012Metric"
 			(at 93.98 87.63 0)
 			(hide yes)
@@
 			)
 		)
-		(property "Description" "Polarized capacitor, small symbol"
+		(property "Description" "Unpolarized capacitor, small symbol"
 			(at 93.98 87.63 0)
 			(hide yes)
@@
 		(lib_id "Transistor_FET:NTMFS016N06CT1G")
 		(at 140.97 102.87 0)
-		(mirror x)
 		(unit 1)
 		(body_style 1)
@@
 		)
 		(property "Footprint" "Package_SON:Infineon_PG-TDSON-8_6.15x5.15mm"
-			(at 146.05 100.965 0)
+			(at 146.05 104.775 0)
 			(hide yes)
 			(show_name no)
@@
 		)
 		(property "Datasheet" "https://www.onsemi.cn/download/data-sheet/pdf/ntmfs015n10mcl-d.pdf"
-			(at 146.05 99.06 0)
+			(at 146.05 106.68 0)
 			(hide yes)
 			(show_name no)

Commit message: Surely i didnt miss anything else on the schematc...
Parts:
- added C304, C305, C306: 100n, Capacitor_SMD:C_0603_1608Metric, symbol Device:C_Small
- added C307, C308, C309, C310, C311, C312: (no value), Capacitor_SMD:C_0805_2012Metric, symbol Device:C_Small
- added D301, D302, D303, D304, D305, D306: 1N4148WS, Diode_SMD:D_SOD-323, symbol Diode:1N4148WS
- added R310, R311, R312, R313, R314, R315: 10, Resistor_SMD:R_0603_1608Metric, symbol Device:R_Small
- added R316, R317, R318, R319, R320, R321: (no value), Resistor_SMD:R_0805_2012Metric, symbol Device:R_Small
- C301, C302, C303: value 1u -> 2.2u
- R309: value 4m -> 5m
Connections:
- net GHS2: now also D304.1 (K)
- net GHS3: now also D305.1 (K)
- net GLS1: now also D301.1 (K)
- net GLS2: now also D303.1 (K)
- net GLS3: now also D306.1 (K)
- net GND: now also C301.2, C302.2, C303.2, C304.2, C305.2, C306.2
- net U: now also C308.1, R316.1
- net V: now also C310.1, R318.1
- net VBUS: now also C304.1, C305.1, C306.1, C307.1, C309.1, C311.1
- net W: now also C312.1, R320.1
- net at JP301.2 (B), JP302.1 (A), Q305.1 (S)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: now also R319.1; no longer C302.2
- net at Q301.4 (G), R301.2, TP301.1: now also R311.2
- net at Q305.4 (G), R305.2, TP308.1: now also R312.2
- net at Q303.4 (G), R303.2, TP303.1: now also R314.2
- net at JP301.1 (A), Q304.1 (S), Q304.2 (S)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: now also R317.1; no longer C301.2
- net at Q306.4 (G), R306.2, TP309.1: now also R315.2
- net at JP302.2 (B), Q306.1 (S), Q306.2 (S)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: now also R321.1; no longer C303.2
- net at Q304.4 (G), R304.2, TP307.1: now also R310.2
- net at Q302.4 (G), R302.2, TP302.1: now also R313.2
- new net: C307.2, R316.2
- new net: C309.2, R318.2
- new net: D301.2 (A), R310.1
- new net: D303.2 (A), R312.1
- new net: C310.2, R319.2
- new net: C311.2, R320.2
- new net: C308.2, R317.2
- new net: D305.2 (A), R314.1
- new net: D306.2 (A), R315.1
- new net: C312.2, R321.2
- new net: D302.2 (A), R311.1
- new net: D304.2 (A), R313.1
Other:
- moved on the sheet: R301, R302, R303, R304, R305, R306, TP301, TP307

Commit message: Updated schematic started on layout for motor PCB
Parts:
- C301, C302, C303: footprint Capacitor_SMD:C_0805_2012Metric -> Capacitor_SMD:C_1210_3225Metric
Connections:
- net GHS1: now also D302.1 (K)
Other:
- moved on the sheet: C305, C307, C308, C309, C310, C311, C312, D301, D302, D303, D304, D305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

Commit message: 20/10-2026
Parts:
- added C313, C314, C315, C316, C317, C318: C_Small, symbol Device:C_Small
- JP301, JP302: footprint Jumper:SolderJumper-2_P1.3mm_Open_Pad1.0x1.5mm -> MOTOR_PCB:SolderJumper-2P_Open_Pad_4.5x2.5mm
Connections:
- net GND: now also C313.2, C314.2, C315.2, C316.2, C317.2, C318.2
- net at Q301.4 (G), R301.2, R311.2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: now also C313.1
- net at Q305.4 (G), R305.2, R312.2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: now also C315.1
- net at Q303.4 (G), R303.2, R314.2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: now also C318.1
- net at Q306.4 (G), R306.2, R315.2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: now also C317.1
- net at Q304.4 (G), R304.2, R310.2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: now also C314.1
- net at Q302.4 (G), R302.2, R313.2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: now also C316.1
Other:
- moved on the sheet: C302, D303, R312, TP310, TP311, TP312

Commit message: 23-10-2026
Parts:
- C313, C314, C315, C316, C317, C318: footprint (none) -> Capacitor_SMD:C_0805_2012Metric
Connections:
- net GND: no longer C313.2, C314.2, C315.2, C316.2, C317.2, C318.2
- net U: now also C313.2
- net V: now also C316.2
- net W: now also C318.2
- net at JP301.1 (A), Q304.1 (S), Q304.2 (S)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: now also C314.2
- net at JP301.2 (B), JP302.1 (A), Q305.1 (S)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: now also C315.2
- net at JP302.2 (B), Q306.1 (S), Q306.2 (S)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: now also C317.2
Other:
- moved on the sheet: C315
