File: Motor_PCB/Motor_PCB.kicad_pcb (KiCad board)
At the start: 4 copper layers, 55 x 100 mm, 262 parts, among them J101 Conn_01x05, J102 Conn_01x03_Pin, J104 Minifit 2x3, J105 Conn_01x06, J106 Conn_01x06, J201 Micro Match, Q101 MMBT3904, Q102 MMBT3904, Q103 MMBT3904, Q301 TPH4R50ANH1, Q302 TPH4R50ANH1, Q303 TPH4R50ANH1, Q304 TPH4R50ANH1, Q305 TPH4R50ANH1, Q306 TPH4R50ANH1, Q401 BC846, Q402 TPH4R50ANH1, Q403 TPH4R50ANH1, Q404 2N7002, Q405 2N7002, Q406 BC856, U201 STSPIN32G4, U202 L78L05_SOT89, U203 LMT86DCK, U204 DRV5053, U205 DRV5053, U401 VOM1271T, U402 TCAN1043H, Y201 ABM3BAIG

Commit message: 20/10-2026
Parts:
- added J103: Conn_01x05, MOTOR_PCB:1411976, F.Cu at (266.9, 23.0)
- JP301, JP302: footprint Jumper:SolderJumper-2_P1.3mm_Open_Pad1.0x1.5mm -> MOTOR_PCB:SolderJumper-2P_Open_Pad_4.5x2.5mm; moved to B.Cu
- R204, R209, R216: value 10k -> 5.1k
- R205, R210, R217: value 100k -> 120k
- R206, R211, R218: value 6.2k -> 4.7k
- R245, R246, R247: value 11k -> 33k
- moved R210 363.8 mm to (376.7, -89.7)
- moved R211 363.8 mm to (376.7, -87.2)
- moved R216 363.8 mm to (376.7, -74.7)
- moved R217 363.8 mm to (376.7, -72.2)
- moved R218 363.8 mm to (376.7, -69.7)
- moved C212 363.8 mm to (364.6, -74.7)
- moved C213 363.8 mm to (364.6, -72.2)
- moved C223 363.8 mm to (368.6, -82.2)
- moved R204 363.8 mm to (372.6, -77.2)
- moved R205 363.8 mm to (372.6, -74.7)
- moved R206 363.8 mm to (372.6, -72.2)
- moved R209 363.8 mm to (372.6, -64.6)
- moved TP201 363.8 mm to (364.4, -61.6)
- moved TP202 363.8 mm to (364.4, -58.0)
- moved TP209 363.8 mm to (371.5, -61.6)
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Connections:
- net /IO/CANH renamed /CANH
- net /IO/CANL renamed /CANL
- net /IO/HEARTBEAT_IN renamed /heatbeat
- C232 pad 1: Net-(U204-VCC) -> +5V
- C232 pad 2: Net-(U204-GND) -> GND
- C233 pad 2: Net-(U204-GND) -> GND
- C234 pad 1: Net-(U205-VCC) -> +5V
- C234 pad 2: Net-(U205-GND) -> GND
- C235 pad 2: Net-(U205-GND) -> GND
- U204 pad 1: Net-(U204-VCC) -> +5V
- U204 pad 3: Net-(U204-GND) -> GND
- U205 pad 1: Net-(U205-VCC) -> +5V
- U205 pad 3: Net-(U205-GND) -> GND
Routing:
- net /MOTOR_W: track 0.00 -> 24.2 mm
- net /MOTOR_U: track 0.00 -> 20.1 mm
- net /MOTOR_V: track 0.00 -> 20.1 mm
- net /Inverter/V_SHUNT_V_N: track 0.00 -> 2.14 mm, vias 0 -> 1
- net /Inverter/V_SHUNT_V_P: track 0.00 -> 1.84 mm, vias 0 -> 1
Other:
- board size 55 x 100 mm -> 62 x 110 mm
- copper layers 4 -> 2

Commit message: 23-10-2026
Parts:
- added C236: 100n, Capacitor_SMD:C_0603_1608Metric, F.Cu at (201.9, 63.9)
- added C237: 10u, Capacitor_SMD:C_0603_1608Metric, F.Cu at (209.3, 67.6)
- added C313: C_Small, Capacitor_SMD:C_0805_2012Metric, B.Cu at (173.2, 92.1)
- added C314: C_Small, Capacitor_SMD:C_0805_2012Metric, B.Cu at (173.1, 101.1)
- added C315: C_Small, Capacitor_SMD:C_0805_2012Metric, B.Cu at (184.4, 101.6)
- added C316: C_Small, Capacitor_SMD:C_0805_2012Metric, B.Cu at (184.4, 91.8)
- added C317: C_Small, Capacitor_SMD:C_0805_2012Metric, B.Cu at (195.6, 101.7)
- added C318: C_Small, Capacitor_SMD:C_0805_2012Metric, B.Cu at (195.5, 91.6)
- added J203: Conn_01x04, Connector_PinHeader_2.54mm:PinHeader_1x04_P2.54mm_Vertical, F.Cu at (160.2, 112.0)
- added JP201: SolderJumper_2_Open, Jumper:SolderJumper-2_P1.3mm_Open_Pad1.0x1.5mm, B.Cu at (191.1, 70.8)
- added Q201: AO3400A, Package_TO_SOT_SMD:SOT-23, F.Cu at (199.9, 60.2)
- added R257: 30k, Resistor_SMD:R_0603_1608Metric, F.Cu at (203.9, 61.0)
- added R258: 100k, Resistor_SMD:R_0603_1608Metric, F.Cu at (207.2, 61.0)
- added R259: 1k, Resistor_SMD:R_0603_1608Metric, F.Cu at (209.3, 64.3)
- added R260: 1k, Resistor_SMD:R_0603_1608Metric, F.Cu at (201.9, 67.7)
- added TP225: TestPoint, TestPoint:TestPoint_Pad_D1.5mm, F.Cu at (155.1, 115.1)
- added TP227: TestPoint, TestPoint:TestPoint_Pad_D1.5mm, F.Cu at (157.8, 115.1)
- added U207: LM358, Package_SO:SOIC-8_3.9x4.9mm_P1.27mm, F.Cu at (205.6, 66.0)
- C228, R228, R230: moved to B.Cu
- Q404: value 2N7002 -> AO3400A
- R242, R243, R244: value 1.5k -> 3k
- moved C308 253.4 mm to (165.1, 100.5)
- moved R316 253.4 mm to (165.1, 96.8)
- moved C307 253.4 mm to (165.1, 93.1)
- moved R317 253.4 mm to (165.1, 104.3)
- moved R252 252.2 mm to (151.9, 115.5)
- moved R210 245.9 mm to (173.9, 49.4), turned to 90 degrees
- moved R211 243.1 mm to (175.6, 49.4), turned to -90 degrees
- moved R216 240.2 mm to (168.8, 45.8)
- moved R218 239.9 mm to (167.8, 48.4), turned to -90 degrees
- moved R217 239.6 mm to (169.5, 48.4), turned to 90 degrees
- moved C223 236.7 mm to (171.2, 48.5), turned to 90 degrees
- moved R251 235.9 mm to (161.0, 115.2), turned to 180 degrees
- moved TP209 230.5 mm to (170.7, 51.4)
- moved R244 229.9 mm to (165.8, 75.9), turned to 180 degrees
- moved R204 228.1 mm to (181.3, 47.0), turned to 180 degrees
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Connections:
- C210 pad 1: +5V -> Net-(Q201-D)
- C211 pad 1: +5V -> Net-(Q201-D)
- C235 pad 1: /STSpin/EOS2 -> GND
- C235 pad 2: GND -> Net-(U201A-PA4)
- R253 pad 1: /STSpin/V_W_meas -> /STSpin/V_U_meas
- U201 pad 10: /STSpin/V_V_meas -> /STSpin/AD_VBUS
- U201 pad 12: /STSpin/AD_VBUS_IN -> /STSpin/V_V_meas
- U201 pad 13: /STSpin/AD_VBUS -> /STSpin/V_W_meas
- U201 pad 51: /LED_WHITE -> /ENA_INRUSH
- U201 pad 53: /ENA_INRUSH -> /LED_WHITE
- U201 pad 9: /STSpin/V_U_meas -> /STSpin/AD_VBUS_IN
- U202 pad 1: +5V -> Net-(Q201-D)
Routing:
- net +5V: track 0.00 -> 148.1 mm, vias 0 -> 5
- net +3V3: track 2.28 -> 89.3 mm, vias 0 -> 7
- net VBUS: track 0.00 -> 83.9 mm, vias 0 -> 2
- net /HALL_W: track 0.00 -> 72.7 mm, vias 0 -> 2
- net /HALL_V: track 0.00 -> 68.1 mm, vias 0 -> 2
- net VBUS_IN: track 0.00 -> 67.8 mm
- net GND: track 0.00 -> 65.5 mm, vias 0 -> 78
- net /HALL_U: track 0.00 -> 61.6 mm, vias 0 -> 2
- net /CANL: track 0.00 -> 55.7 mm
- net /CANH: track 0.00 -> 49.1 mm
- net /LED_WHITE: track 0.00 -> 47.5 mm
- net /LED_GREEN: track 0.00 -> 47.4 mm
- net /LED_RED: track 0.00 -> 46.4 mm
- net /AD_TEMP: track 0.00 -> 41.2 mm, vias 0 -> 1
- net /STSpin/PROG_RX: track 0.00 -> 36.6 mm
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- added copper zone on B.Cu, net GND
- added copper zone on F.Cu, net GND
- added copper zone on In1.Cu, net GND
- added copper zone on In2.Cu, net GND
- added copper zone on F.Cu, net VBUS
Other:
- copper layers 2 -> 4
- board text added: "ADD mounting options"
- board text added: "Add silkscreen to all Testpoints - Assume it is not you measuring!"
- board text added: "Find webpage for Heat source"
