File: Motor_PCB/STSpin.kicad_sch (KiCad schematic)
At the start: 1 part, among them U1 STSPIN32G4

Commit message: Schematics mostly done
Parts:
- added C201, C202, C203: 1u, symbol Device:C_Small
- added C204, C209, C210, C215, C217, C219: 10u, symbol Device:C_Small
- added C205, C206: 24p, Capacitor_SMD:C_0603_1608Metric, symbol Device:C_Small
- added C207: 10n, Capacitor_SMD:C_0603_1608Metric, symbol Device:C_Small
- added C208, C229: 220n, symbol Device:C_Small
- added C211, C216, C218, C220, C221, C224: 100n, symbol Device:C_Small
- added C212, C213, C214, C222, C223, C230: 47n, Capacitor_SMD:C_0603_1608Metric, symbol Device:C_Small
- added C225, C226, C227: 1n, symbol Device:C_Small
- added C228: 1u, Capacitor_SMD:C_0603_1608Metric, symbol Device:C_Small
- added C231: 100n, Capacitor_SMD:C_0603_1608Metric, symbol Device:C_Small
- added D201: STPS1H100A, symbol Device:D_Schottky
- added D202, D203: MM3Z56VB, Diode_SMD:D_SMA, symbol Diode:MM3Zxx
- added D204: PESD5V2S2UT, Package_TO_SOT_SMD:SOT-23, symbol Device:D_Zener_Dual_CommonAnode_KKA
- added J201: Micro Match, MOTOR_PCB:CONN6_7-188275-6_TEC, symbol Connector_Generic:Conn_02x03_Counter_Clockwise
- added L201: 18u, symbol Device:L_Small
- added R201, R203: 0, symbol Device:R_Small
- added R202: 10k, Resistor_SMD:R_0603_1608Metric, symbol Device:R_Small
- added R204, R207, R208, R209, R216, R230: 100k, Resistor_SMD:R_0603_1608Metric, symbol Device:R_Small
- added R205, R210, R212, R213, R217: 220k, Resistor_SMD:R_0603_1608Metric, symbol Device:R_Small
- added R206, R211, R214, R215, R218: 12k, Resistor_SMD:R_0603_1608Metric, symbol Device:R_Small
- added R219, R220, R221, R222: 10k, symbol Device:R_Small
- added R223: 4.7k, symbol Device:R_Small
- added R224: 10, symbol Device:R_Small
- added R225, R226, R227: 100, symbol Device:R_Small
- added R228: 15k, Resistor_SMD:R_0603_1608Metric, symbol Device:R_Small
- added R229, R240: 120, Resistor_SMD:R_0603_1608Metric, symbol Device:R_Small
- added R231, R232, R233, R237, R238, R239: 22k, Resistor_SMD:R_0603_1608Metric, symbol Device:R_Small
- added R234, R235, R236, R242, R243, R244: 1.5k, Resistor_SMD:R_0603_1608Metric, symbol Device:R_Small
- added R241: 470k, Resistor_SMD:R_0603_1608Metric, symbol Device:R_Small
- added R245, R246, R247: 11k, Resistor_SMD:R_0603_1608Metric, symbol Device:R_Small
- added R248: 10K, Resistor_SMD:R_0603_1608Metric, symbol Device:R_Small
- added R249: 22K, Resistor_SMD:R_0603_1608Metric, symbol Device:R_Small
- added R250: 1k, symbol Device:R_Small
- added TP201, TP202, TP203, TP204, TP205, TP206, TP207, TP208, TP209, TP210, TP211, TP212, TP213, TP214, TP215, TP216, TP217, TP218, TP219, TP220, TP221, TP222, TP223, TP224: TestPoint, TestPoint:TestPoint_Pad_D1.5mm, symbol Connector:TestPoint
- added U202: L78L05_SOT89, Package_TO_SOT_SMD:SOT-89-3, symbol Regulator_Linear:L78L05_SOT89
- added U203: LMT86DCK, Package_TO_SOT_SMD:SOT-353_SC-70-5, symbol Sensor_Temperature:LMT86DCK
- added Y201: ABM3BAIG, Crystal:Crystal_SMD_5032-4Pin_5.0x3.2mm, symbol Device:Crystal_GND24
- renumbered U1 to U201
Connections:
- net VCC: now also U201.63 (VCC), C209.1, R201.2, R203.1, U202.3 (IN); no longer U201.61 (VM)
- net +3V3: now reaches U201.1 (REG3V3/VDD)
- net +3V3: now also U201.2 (VBAT), U201.26 (VREF+), U201.27 (VDDA), C215.1, C216.1, C217.1, C218.1, C219.1, C220.1, C221.1, C231.2, J201.5 (Pin_5), R202.2, R219.1, R220.1, R221.1, R222.1, R231.1, R232.1, R233.1, R249.1, TP205.1, TP206.1, TP207.1, TP208.1, U203.4 (V_{DD}), U203.5 (V_{DD})
- net GND: now reaches U201.32 (PGND)
- net GND: now also U201.65 (VSS), C204.2, C205.2, C206.2, C207.1, C208.2, C209.2, C210.2, C211.2, C212.2, C213.2, C214.2, C215.2, C216.2, C217.2, C218.2, C219.2, C220.2, C221.2, C222.2, C223.2, C224.2, C225.2, C226.2, C227.2, C228.1, C229.2, C230.1, C231.1, D201.2 (A), D202.2 (A), D203.2 (A), D204.3 (A), J201.2 (Pin_2), R206.1, R211.1, R214.2, R215.2, R218.1, R230.1, R237.2, R238.2, R239.2, R241.1, R248.2, U202.2 (GND), U203.1 (GND), U203.2 (GND), Y201.2 (G), Y201.4 (G)
- net V_V_meas: now reaches U201.10 (PC1)
- net V_V_meas: now also C213.1, R210.1, R211.2, TP202.1
- net V_W_meas: now reaches U201.11 (PC2)
- net V_W_meas: now also C223.1, R217.1, R218.2, TP209.1
- net AD_VBUS_IN: now reaches U201.12 (PC3)
- net AD_VBUS_IN: now also C214.1, R212.2, R214.1, TP203.1
- net AD_VBUS: now reaches U201.13 (PA0)
- net AD_VBUS: now also C222.1, R213.2, R215.1, TP204.1
- net OP1_Pos: now reaches U201.14 (PA1)
- net OP1_Pos: now also R231.2, R234.1, R237.1, TP216.1
- net OP1_Out: now reaches U201.15 (PA2)
- net OP1_Out: now also R245.1, TP219.1
- net OP1_Neg: now reaches U201.16 (PA3)
- net OP1_Neg: now also R242.1, R245.2
- net AD_TEMP_mcu: now reaches U201.17 (PA4)
- net AD_TEMP_mcu: now also R223.2, TP210.1
- net LED_GREEN: now reaches U201.18 (PA5)
- net OP2_Out: now reaches U201.19 (PA6)
- net OP2_Out: now also R246.1, TP222.1
- net OP2_Pos: now reaches U201.20 (PA7)
- net OP2_Pos: now also R232.2, R235.1, R238.1, TP217.1
- net AD_TEMP_FET: now reaches U201.21 (PC4)
- net AD_TEMP_FET: now also C230.2, R250.2, TP224.1
- net OP2_Neg: now reaches U201.22 (PC5)
- net OP2_Neg: now also R243.1, R246.2
- net OP3_Pos: now reaches U201.23 (PB0)
- net OP3_Pos: now also R233.2, R236.1, R239.1, TP218.1
- net OP3_Out: now reaches U201.24 (PB1)
- net OP3_Out: now also R247.1, TP223.1
- net OP3_Neg: now reaches U201.25 (PB2)
- net OP3_Neg: now also R244.1, R247.2
- net GLS1: now reaches U201.29 (GLS1)
- net WAKE: now reaches U201.3 (PC13)
- net GLS2: now reaches U201.30 (GLS2)
- net GLS3: now reaches U201.31 (GLS3)
- net at U201.35 (BOOT3): now also C203.2
- net PHASE_W: now reaches U201.36 (OUT3)
- net PHASE_W: now also C203.1
- net GHS3: now reaches U201.37 (GHS3)
- net at U201.38 (BOOT2): now also C202.2
- net PHASE_V: now reaches U201.39 (OUT2)
- net PHASE_V: now also C202.1
- net CAN_STB: now reaches U201.4 (PC14)
- net GHS2: now reaches U201.40 (GHS2)
- net at U201.41 (BOOT1): now also C201.2
- net PHASE_U: now reaches U201.42 (OUT1)
- net PHASE_U: now also C201.1
- net GHS1: now reaches U201.43 (GHS1)
- net CAN_FAULT: now reaches U201.44 (PA8)
- net PROG_TX: now reaches U201.45 (PA9)
- net PROG_TX: now also D204.1 (K), R240.2, R241.2, TP221.1
- net PROG_RX: now reaches U201.46 (PA10)
- net PROG_RX: now also D204.2 (K), R228.1, R229.2, TP215.1
- net CAN_RX: now reaches U201.47 (PA11)
- net CAN_TX: now reaches U201.48 (PA12)
- net SWD_IO: now reaches U201.49 (PA13)
- net SWD_IO: now also J201.1 (Pin_1)
- net CAN_ENA: now reaches U201.5 (PC15)
- net SWD_CLK: now reaches U201.50 (PA14)
- net SWD_CLK: now also J201.3 (Pin_3)
- net LED_BLUE: now reaches U201.51 (PA15)
- net at U201.52 (SCREF): now also C229.1, R248.1, R249.2
- net ENA_INRUSH: now reaches U201.53 (PD2)
- net SWO: now reaches U201.54 (PB3)
- net SWO: now also J201.6 (Pin_6)
- net LED_RED: now reaches U201.56 (PB5)
- net HALL_U_mcu: now reaches U201.57 (PB6)
- net HALL_U_mcu: now also C225.1, R220.2, R225.2, TP211.1
- net HALL_V_mcu: now reaches U201.58 (PB7)
- net HALL_V_mcu: now also C226.1, R221.2, R226.2, TP212.1
- net HALL_W_mcu: now reaches U201.59 (PB8)
- net HALL_W_mcu: now also C227.1, R222.2, R227.2, TP213.1
- net at U201.6 (PF0): now also C205.1, Y201.1
- net HEARTBEAT: now reaches U201.60 (PB9)
- net SW: now reaches U201.62 (SW)
- net SW: now also D201.1 (K), L201.1
- net at U201.64 (REGIN): now also R203.2
- net at U201.7 (PF1): now also C206.1, Y201.3
- net ~{RST}: now reaches U201.8 (PG10)
- net ~{RST}: now also C207.2, J201.4 (Pin_4), R202.1
- net V_U_meas: now reaches U201.9 (PC0)
- net V_U_meas: now also C212.1, R205.1, R206.2, TP201.1
- new net: C224.1, R219.2, R223.1, R224.2
- new net: C204.1, L201.2, R201.1
- new net: R204.1, R205.2
- new net: R229.1, TP214.1
- new net: D203.1 (K), R208.2, R213.1
- new net: R216.1, R217.2
- new net: R240.1, TP220.1
- new net: D202.1 (K), R207.2, R212.1
- new net: R250.1, U203.3 (OUT)
- new net: R209.1, R210.2
- new net +5V: C210.1, C211.1, U202.1 (OUT)
- new net AD_TEMP: R224.1
- new net HALL_U: R225.1
- new net HALL_V: R226.1
- new net HALL_W: R227.1
- new net MOTOR_U: R204.2
- new net MOTOR_V: R209.2
- new net MOTOR_W: R216.2
- new net PROG_BOOT: C228.2, R228.2, R230.2
- new net VBUS: C208.1, R208.1, U201.61 (VM)
- new net VBUS_IN: R207.1
- new net V_SHUNT_U_N: R242.2
- new net V_SHUNT_U_P: R234.2
- new net V_SHUNT_V_N: R243.2
- new net V_SHUNT_V_P: R235.2
- new net V_SHUNT_W_N: R244.2
- new net V_SHUNT_W_P: R236.2
- no-connect marks 0 -> 2
Other:
- note added: "+"
- note added: "-"
- note added: "36.15mV/V"
- note added: "5V LDO"
- note added: "8MHz"
- note added: "CON_PROG_RX"
- note added: "CON_PROG_TX"
- note added: "Current Shunt AMP"
- note added: "Decoupling"
- note added: "HALL"
- note added: "HALL CAN BE MOVED TO TIM3 ON PB4, PB5 AND PB0 (AT THE COST OF (OP3)"
- note added: "Motor Temp"
- note added: "PB8 is used for HALL!"
- note added: "PROG 6-pin"
- note added: "PROG_BOOT!"
- note added: "Phase Measurement"
- note added: "Place close to mcu pin"
- note added: "Shunt amp phaes U"
- note added: "Shunt amp phaes V"
- note added: "Shunt amp phaes W"
- note added: "Supply Measurement"
- note added: "UART"
- note added: "VBAT"
- note added: "VDD"
- note added: "VDDA"
- note added: "VREF+"
- moved on the sheet: U201A, U201B

Commit message: Fixed some Schematic mistakes
- Fixed mirroers FETS
- Added voltage divider to TCAN INH
- fixed other minor mistakes
Parts:
- added FB201: FerriteBead_Small, Inductor_SMD:L_0603_1608Metric, symbol Device:FerriteBead_Small
- C201, C202, C203, C209, C210, C215, C217, C219: footprint (none) -> Capacitor_SMD:C_0805_2012Metric
- C204, C208, C211, C216, C218, C220, C221, C224, C225, C226, C227, C229: footprint (none) -> Capacitor_SMD:C_0603_1608Metric
- C212, C213, C223: value 47n -> 10n
- R201, R203, R219, R220, R221, R222, R223, R224, R225, R226, R227, R250: footprint (none) -> Resistor_SMD:R_0603_1608Metric
- R204, R209, R216: value 100k -> 10k
- R205, R210, R217: value 220k -> 100k
- R206, R211, R218: value 12k -> 6.2k
- U201: footprint QFN_IN32G4_STM -> MOTOR_PCB:QFN_IN32G4_STM
Connections:
- net +3V3: now also FB201.1; no longer C217.1, C218.1, C219.1, C220.1, TP206.1, TP207.1, U201.26 (VREF+), U201.27 (VDDA)
- net HEARTBEAT: now also U201.28 (PB10); no longer U201.60 (PB9)
- new net +3V3_VDDA: C217.1, C218.1, C219.1, C220.1, FB201.2, TP206.1, TP207.1, U201.26 (VREF+), U201.27 (VDDA)
Other:
- note added: "PB10 HAS TIM1_BKIN"
- note removed: "VDDA"
- moved on the sheet: C217, C218, R201, TP206

Commit message: Surely i didnt miss anything else on the schematc...
Parts:
- D201: footprint (none) -> Diode_SMD:D_SMA
- L201: footprint (none) -> Inductor_SMD:L_APV_ANR4020
Changed lines of the file:
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@@
 			)
 		)
-		(property "Footprint" ""
+		(property "Footprint" "Inductor_SMD:L_APV_ANR4020"
 			(at 210.82 86.36 0)
 			(hide yes)
@@
 			)
 		)
-		(property "Datasheet" ""
+		(property "Datasheet" "https://jlcpcb.com/partdetail/APV-ANR4030T180M/C6808099"
 			(at 210.82 86.36 0)
 			(hide yes)
@@
 		)
 		(property "Value" "STPS1H100A"
-			(at 203.2 85.09 0)
+			(at 191.77 81.28 90)
 			(show_name no)
 			(do_not_autoplace no)
@@
 			)
 		)
-		(property "Footprint" ""
+		(property "Footprint" "Diode_SMD:D_SMA"
 			(at 205.74 81.28 0)
 			(hide yes)

Commit message: Updated schematic started on layout for motor PCB
Parts:
- added C232, C233, C234, C235: 100n, Capacitor_SMD:C_0603_1608Metric, symbol Device:C_Small
- added R251, R252: 10k, Resistor_SMD:R_0603_1608Metric, symbol Device:R_Small
- added R253, R254, R255, R256: 0, Resistor_SMD:R_0603_1608Metric, symbol Device:R_Small
- added U204, U205: DRV5053, Package_TO_SOT_SMD:SOT-23, symbol Sensor_Magnetic:DRV5055A1xDBZxQ1
- D202, D203: footprint Diode_SMD:D_SMA -> Diode_SMD:D_SOD-323F
Connections:
- net LED_GREEN: now also U201.55 (PB4); no longer U201.18 (PA5)
- net V_W_meas: now also R253.1; no longer U201.11 (PC2)
- net AD_TEMP_mcu renamed AD_TEMP_motor
- net AD_TEMP_motor: now also R256.2; no longer U201.17 (PA4)
- new net: C234.1, U205.1 (VCC)
- new net: C234.2, C235.2, U205.3 (GND)
- new net: R252.1, U205.2 (OUT)
- new net: R255.1, R256.1, U201.17 (PA4)
- new net: R251.1, U204.2 (OUT)
- new net: C232.1, U204.1 (VCC)
- new net: C232.2, C233.2, U204.3 (GND)
- new net: R253.2, R254.2, U201.11 (PC2)
- new net EOS1: C233.1, R251.2, U201.18 (PA5)
- new net EOS2: C235.1, R252.2, R254.1, R255.2
- no-connect marks 2 -> 1
Other:
- moved on the sheet: C204, C217, C218, D201, FB201, L201, R201, TP206, U201B

Commit message: 20/10-2026
Parts:
- added J203: Conn_01x04, symbol Connector_Generic:Conn_01x04
- added TP225, TP227: TestPoint, TestPoint:TestPoint_Pad_D1.5mm, symbol Connector:TestPoint
- R204, R209, R216: value 10k -> 5.1k
- R205, R210, R217: value 100k -> 120k
- R206, R211, R218: value 6.2k -> 4.7k
- R245, R246, R247: value 11k -> 33k
- R253, R255: now not fitted
Connections:
- net +5V: now also C232.1, C234.1, U204.1 (VCC), U205.1 (VCC), J203.1 (Pin_1)
- net EOS1: now also J203.2 (Pin_2), TP227.1
- net EOS2: now also J203.3 (Pin_3), TP225.1
- net GND: now also C232.2, C233.2, C234.2, C235.2, U204.3 (GND), U205.3 (GND), J203.4 (Pin_4)
Other:
- note added: "36.21 mV/V"
- note added: "Add start up timer"
- moved on the sheet: C201, C202, C203, C205, C206, C207, C208, C215, C216, C217, C218, C219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

Commit message: 23-10-2026
Parts:
- added C236: 100n, Capacitor_SMD:C_0603_1608Metric, symbol Device:C_Small
- added C237: 10u, Capacitor_SMD:C_0603_1608Metric, symbol Device:C_Small
- added JP201: SolderJumper_2_Open, Jumper:SolderJumper-2_P1.3mm_Open_Pad1.0x1.5mm, symbol Jumper:SolderJumper_2_Open
- added Q201: AO3400A, Package_TO_SOT_SMD:SOT-23, symbol Transistor_FET:AO3400A
- added R257: 30k, Resistor_SMD:R_0603_1608Metric, symbol Device:R_Small
- added R258: 100k, Resistor_SMD:R_0603_1608Metric, symbol Device:R_Small
- added R259, R260: 1k, Resistor_SMD:R_0603_1608Metric, symbol Device:R_Small
- added U207: LM358, Package_SO:SOIC-8_3.9x4.9mm_P1.27mm, symbol Amplifier_Operational:LM358
- J201: now not fitted
- J203: footprint (none) -> Connector_PinHeader_2.54mm:PinHeader_1x04_P2.54mm_Vertical
- R242, R243, R244: value 1.5k -> 3k
Connections:
- net +5V: now also Q201.2 (S); no longer C210.1, C211.1, U202.1 (OUT)
- net AD_VBUS: now also U201.10 (PC1); no longer U201.13 (PA0)
- net AD_VBUS_IN: now also U201.9 (PC0); no longer U201.12 (PC3)
- net ENA_INRUSH: now also U201.51 (PA15); no longer U201.53 (PD2)
- net EOS2: no longer C235.1
- net GND: now also C235.1, C236.2, C237.2, R258.2, U207.4 (V-); no longer C235.2
- net HALL_W_mcu: now also JP201.2 (B)
- net LED_BLUE: now also U201.53 (PD2); no longer U201.51 (PA15)
- net PROG_BOOT: now also JP201.1 (A)
- net VCC: now also C236.1, U207.8 (V+)
- net V_U_meas: now also R253.1; no longer U201.9 (PC0)
- net V_V_meas: now also U201.12 (PC3); no longer U201.10 (PC1)
- net V_W_meas: now also U201.13 (PA0); no longer R253.1
- net at R255.1, R256.1, U201.17 (PA4): now also C235.2
- new net: C210.1, C211.1, Q201.3 (D), R257.1, R259.1, U202.1 (OUT)
- new net: Q201.1 (G), R260.1
- new net: R260.2, U207.1
- new net RC_10m: C237.1, R259.2, U207.3 (+)
- new net Ref_3V8_in: R257.2, R258.1, U207.5 (+)
- new net Ref_3V8_out: U207.2 (-), U207.6 (-), U207.7
Other:
- note added: "Add pcb pads you can scratch out... To all power nets"
- note added: "Double check the ADC input caps Sampling buffer"
- note added: "PROG_BOOT Pin (PB8) is used for HALL!"
- note removed: "Add start up timer"
- note removed: "PB8 is used for HALL!"
- moved on the sheet: C210, C211, C235, R218
